File: NUSBIO BOARD/Nusbio1.0.WaveShare.WithLed.SeedStudio/bu/Nusbio1.0.WaveShare.WithLed.SeedStudio.sch (EAGLE design)
At the start: 15 parts

Commit message: board 4017-7Segment v2 on hold, until I received chip 4017B
Parts:
- renumbered RPWR to RPWR_470_O
Changed lines of the file:
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@@
 <part name="LED5" library="adafruit" deviceset="LED" device="SMT1206"/>
 <part name="LPOWER" library="adafruit" deviceset="LED" device="SMT1206"/>
-<part name="RPWR" library="adafruit" deviceset="R-US_" device="R1206"/>
+<part name="RPWR_470_O" library="adafruit" deviceset="R-US_" device="R1206"/>
 <part name="GND4" library="supply1" deviceset="GND" device=""/>
 </parts>
@@
 <instance part="LED5" gate="G$1" x="167.64" y="43.18" rot="R180"/>
 <instance part="LPOWER" gate="G$1" x="139.7" y="15.24" rot="R180"/>
-<instance part="RPWR" gate="G$1" x="132.08" y="33.02" rot="R90"/>
+<instance part="RPWR_470_O" gate="G$1" x="132.08" y="33.02" rot="R90"/>
 <instance part="GND4" gate="1" x="132.08" y="45.72" rot="R180"/>
 </instances>
@@
 </segment>
 <segment>
-<pinref part="RPWR" gate="G$1" pin="2"/>
+<pinref part="RPWR_470_O" gate="G$1" pin="2"/>
 <pinref part="GND4" gate="1" pin="GND"/>
 <wire x1="132.08" y1="38.1" x2="132.08" y2="43.18" width="0.1524" layer="91"/>
@@
 <segment>
 <pinref part="LPOWER" gate="G$1" pin="C"/>
-<pinref part="RPWR" gate="G$1" pin="1"/>
+<pinref part="RPWR_470_O" gate="G$1" pin="1"/>
 <wire x1="139.7" y1="20.32" x2="132.08" y2="27.94" width="0.1524" layer="91"/>
 </segment>
