File: EXTENSIONS/Analog/Clock Module Timer 555 -Simplified/bu/NoLogo/Clock Extension.brd (EAGLE design)
At the start: 28 x 48 mm, 8 parts, among them T555_CLOCK NE555N, X1 USB-A

Commit message: Update/create Clock Module Time 555 -Simplified
Parts:
- moved C1_33UF 0.50 mm to (11.0, 44.5)
- moved LED_OUTPUT 0.50 mm to (21.2, 43.5)
- moved R2_POT_10K 0.50 mm to (16.0, 22.5)
- moved T555_CLOCK 0.50 mm to (9.50, 34.0)
Other:
- board text added: "NC"
- board text removed: "OUT_R"
Changed lines of the file:
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@@
 <text x="7.5" y="17" size="1.016" layer="25">GND</text>
 <text x="14.4" y="53.2" size="1.016" layer="25" rot="R90">VCC</text>
-<text x="19.5" y="53.7" size="1.016" layer="25" rot="R270" align="center">OUT_R</text>
+<text x="19.5" y="53.7" size="1.016" layer="25" rot="R270" align="center">NC</text>
 <text x="16" y="49.5" size="1.6764" layer="25" align="center">CLOCK MODULE</text>
-<text x="6.5" y="44" size="1.27" layer="25">+</text>
-<text x="23.5" y="45.2" size="1.27" layer="25">+</text>
+<text x="6.5" y="44.5" size="1.27" layer="25">+</text>
+<text x="23.5" y="45.7" size="1.27" layer="25">+</text>
 </plain>
 <attributes>
@@
 </autorouter>
 <elements>
-<element name="C1_33UF" library="adafruit" package="C025-030X050" value="" x="11" y="44" smashed="yes" rot="R180">
-<attribute name="NAME" x="11.3" y="41.2" size="1.016" layer="25" ratio="10" rot="R180" align="center"/>
-<attribute name="VALUE" x="13.286" y="47.048" size="1.27" layer="27" ratio="10" rot="R180"/>
+<element name="C1_33UF" library="adafruit" package="C025-030X050" value="" x="11" y="44.5" smashed="yes" rot="R180">
+<attribute name="NAME" x="11.3" y="41.7" size="1.016" layer="25" ratio="10" rot="R180" align="center"/>
+<attribute name="VALUE" x="13.286" y="47.548" size="1.27" layer="27" ratio="10" rot="R180"/>
 </element>
 <element name="X1" library="adafruit" package="MOLEX_480371000" value="USB-A" x="16" y="14.4" smashed="yes">
 <attribute name="VALUE" x="14.46" y="11.05" size="1.016" layer="27" font="vector"/>
 </element>
-<element name="T555_CLOCK" library="linear" package="DIL08" value="NE555N" x="9.5" y="33.5" smashed="yes" rot="R270">
-<attribute name="VALUE" x="8.865" y="37.056" size="1.27" layer="27" ratio="10" rot="R270"/>
+<element name="T555_CLOCK" library="linear" package="DIL08" value="NE555N" x="9.5" y="34" smashed="yes" rot="R270">
+<attribute name="VALUE" x="8.865" y="37.556" size="1.27" layer="27" ratio="10" rot="R270"/>
 </element>
 <element name="JP1" library="pinhead" package="1X04" value="" x="15.5" y="58" smashed="yes">
@@
 </element>
 <element name="R_1.2K_1" library="adafruit" package="R1206" value="" x="25.5" y="29" smashed="yes" rot="R90">
-<attribute name="NAME" x="24" y="26.5" size="1.016" layer="25" rot="R90"/>
+<attribute name="NAME" x="24" y="26" size="1.016" layer="25" rot="R90"/>
 <attribute name="VALUE" x="27.913" y="27.603" size="1.27" layer="27" rot="R90"/>
 </element>
-<element name="R2_POT_10K" library="SparkFun-Electromechanical" package="TRIM_POT_PTH" value="" x="16" y="23" smashed="yes" rot="R180">
-<attribute name="NAME" x="16.5" y="27.3" size="1.016" layer="25" rot="R180" align="center"/>
-<attribute name="VALUE" x="12.825" y="23" size="0.6096" layer="27" rot="R180"/>
-</element>
-<element name="LED_OUTPUT" library="adafruit" package="1206" value="" x="21.2" y="43" smashed="yes" rot="R270">
-<attribute name="VALUE" x="18.66" y="44.27" size="1.27" layer="27" rot="R270"/>
+<element name="R2_POT_10K" library="SparkFun-Electromechanical" package="TRIM_POT_PTH" value="" x="16" y="22.5" smashed="yes" rot="R180">
+<attribute name="NAME" x="16.5" y="26.8" size="1.016" layer="25" rot="R180" align="center"/>
+<attribute name="VALUE" x="12.825" y="22.5" size="0.6096" layer="27" rot="R180"/>
+</element>
+<element name="LED_OUTPUT" library="adafruit" package="1206" value="" x="21.2" y="43.5" smashed="yes" rot="R270">
+<attribute name="VALUE" x="18.66" y="44.77" size="1.27" layer="27" rot="R270"/>
 </element>
 <element name="R_1K_3" library="adafruit" package="R1206" value="" x="25.5" y="37" smashed="yes" rot="R90">
@@
 <contactref element="JP1" pad="1"/>
 <contactref element="R_1K_3" pad="1"/>
-<wire x1="12.27" y1="44" x2="11.69" y2="58" width="0" layer="19" extent="1-1"/>
-<wire x1="5.69" y1="37.31" x2="12.27" y2="44" width="0" layer="19" extent="1-1"/>
-<wire x1="25.5" y1="35.578" x2="12.27" y2="44" width="0" layer="19" extent="1-1"/>
+<wire x1="12.27" y1="44.5" x2="11.69" y2="58" width="0" layer="19" extent="1-1"/>
+<wire x1="5.69" y1="37.81" x2="12.27" y2="44.5" width="0" layer="19" extent="1-1"/>
+<wire x1="25.5" y1="35.578" x2="12.27" y2="44.5" width="0" layer="19" extent="1-1"/>
 <wire x1="12.5" y1="17" x2="25.5" y2="35.578" width="0" layer="19" extent="1-1"/>
 </signal>
@@
 <contactref element="JP1" pad="2"/>
 <contactref element="R_1.2K_1" pad="2"/>
-<wire x1="13.31" y1="37.31" x2="14.23" y2="58" width="0" layer="19" extent="1-1"/>
-<wire x1="5.69" y1="29.69" x2="13.31" y2="37.31" width="0" layer="19" extent="1-1"/>
-<wire x1="25.5" y1="30.422" x2="13.31" y2="37.31" width="0" layer="19" extent="1-1"/>
+<wire x1="13.31" y1="37.81" x2="14.23" y2="58" width="0" layer="19" extent="1-1"/>
+<wire x1="5.69" y1="30.19" x2="13.31" y2="37.81" width="0" layer="19" extent="1-1"/>
+<wire x1="25.5" y1="30.422" x2="13.31" y2="37.81" width="0" layer="19" extent="1-1"/>
 <wire x1="19.5" y1="17" x2="25.5" y2="30.422" width="0" layer="19" extent="1-1"/>
 </signal>
@@
 <contactref element="R_1.2K_1" pad="1"/>
 <contactref element="R2_POT_10K" pad="3"/>
-<wire x1="13.46" y1="25.54" x2="25.5" y2="27.578" width="0" layer="19" extent="1-1"/>
-<wire x1="13.31" y1="34.77" x2="13.46" y2="25.54" width="0" layer="19" extent="1-1"/>
+<wire x1="13.46" y1="25.04" x2="25.5" y2="27.578" width="0" layer="19" extent="1-1"/>
+<wire x1="13.31" y1="35.27" x2="13.46" y2="25.04" width="0" layer="19" extent="1-1"/>
 </signal>
 <signal name="THRESHOLD">
@@
 <contactref element="C1_33UF" pad="2"/>
 <contactref element="R2_POT_10K" pad="2"/>
-<wire x1="5.69" y1="34.77" x2="9.73" y2="44" width="0" layer="19" extent="1-1"/>
-<wire x1="13.31" y1="32.23" x2="5.69" y2="34.77" width="0" layer="19" extent="1-1"/>
-<wire x1="16" y1="20.46" x2="13.31" y2="32.23" width="0" layer="19" extent="1-1"/>
+<wire x1="5.69" y1="35.27" x2="9.73" y2="44.5" width="0" layer="19" extent="1-1"/>
+<wire x1="13.31" y1="32.73" x2="5.69" y2="35.27" width="0" layer="19" extent="1-1"/>
+<wire x1="16" y1="19.96" x2="13.31" y2="32.73" width="0" layer="19" extent="1-1"/>
 </signal>
 <signal name="TMR555_OUTPUT">
@@
 <contactref element="JP1" pad="3"/>
 <contactref element="LED_OUTPUT" pad="A"/>
-<wire x1="21.2" y1="44.422" x2="16.77" y2="58" width="0" layer="19" extent="1-1"/>
-<wire x1="5.69" y1="32.23" x2="21.2" y2="44.422" width="0" layer="19" extent="1-1"/>
+<wire x1="21.2" y1="44.922" x2="16.77" y2="58" width="0" layer="19" extent="1-1"/>
+<wire x1="5.69" y1="32.73" x2="21.2" y2="44.922" width="0" layer="19" extent="1-1"/>
 </signal>
 <signal name="N$5">
 <contactref element="LED_OUTPUT" pad="C"/>
 <contactref element="R_1K_3" pad="2"/>
-<wire x1="25.5" y1="38.422" x2="21.2" y2="41.578" width="0" layer="19" extent="1-1"/>
+<wire x1="25.5" y1="38.422" x2="21.2" y2="42.078" width="0" layer="19" extent="1-1"/>
 </signal>
 <signal name="TMR555_OUTPUT_REVERSE">
