File: EXTENSIONS/Analog/fCPU/v1.WithProgramCounterAndControllerAsSN74LS42N/fCPU.brd (EAGLE design)
At the start: 97 x 73 mm, 15 parts

Commit message: Update fCPU
Parts:
- removed ADDER_74LS283N: 74LS283N, 74xx-us:DIL16
- removed CONTROLLER_CD4017BE: CD4017, SparkFun-DigitalIC:DIL16
- removed CONTROLLER_INV_SN74LS14: 74LS14N, 74xx-us:DIL14
- removed DISPLAY_DRIVER_74LS47: 74LS47N, 74xx-us:DIL16
- removed REGISTER_1_SN74LS273, REGISTER_2_SN74LS273: 74273N, 74xx-us:DIL20
- added CONTROLLER: 74LS42N, 74xx-us:DIL16
- added CONTROLLER_INV_: 74LS14N, 74xx-us:DIL14
- added DISPLAY_DRIVER: 74LS47N, 74xx-us:DIL16
- added PRG_COUNTER: 74LS90N, 74xx-us:DIL14
- added REGISTER_1, REGISTER_2: 74273N, 74xx-us:DIL20
- moved DIGIT_0_ANODE 41.3 mm to (9.00, 72.0)
- moved R_100O_0 32.1 mm to (17.5, 78.5), turned to 270 degrees
- moved REGISTER_1_CLEAR_CX 19.3 mm to (43.0, 51.0)
- moved REGISTER_2_CLEAR_CX 12.0 mm to (40.0, 58.0)
Connections:
- removed net CTRL_HIGH_1: CONTROLLER_CD4017BE.3, CONTROLLER_INV_SN74LS14.13
- removed net CTRL_HIGH_2: CONTROLLER_CD4017BE.2, CONTROLLER_INV_SN74LS14.11
- removed net CTRL_HIGH_3: CONTROLLER_CD4017BE.4, CONTROLLER_INV_SN74LS14.9
- removed net CTRL_HIGH_4: CONTROLLER_CD4017BE.7, CONTROLLER_INV_SN74LS14.1
- removed net CTRL_HIGH_5: CONTROLLER_CD4017BE.10, CONTROLLER_INV_SN74LS14.3
- removed net CTRL_HIGH_6: CONTROLLER_CD4017BE.1, CONTROLLER_INV_SN74LS14.5
- removed net CTRL_LOW_1: CONTROLLER_INV_SN74LS14.12, REGISTER_1_CLEAR_CX.1
- removed net CTRL_LOW_2: CONTROLLER_INV_SN74LS14.10, REGISTER_2_CLEAR_CX.1
- removed net CTRL_LOW_3: CONTROLLER_INV_SN74LS14.8
- removed net CTRL_LOW_4: CONTROLLER_INV_SN74LS14.2
- removed net CTRL_LOW_5: CONTROLLER_INV_SN74LS14.4
- removed net CTRL_LOW_6: CONTROLLER_INV_SN74LS14.6
- removed net N$10: ADDER_74LS283N.4
- removed net N$11: ADDER_74LS283N.1
- removed net N$12: ADDER_74LS283N.13
- removed net N$13: ADDER_74LS283N.10
- removed net REGISTER_1_OUT_BIT_0: ADDER_74LS283N.5, REGISTER_1_SN74LS273.2
- removed net REGISTER_1_OUT_BIT_1: ADDER_74LS283N.3, REGISTER_1_SN74LS273.5
- removed net REGISTER_1_OUT_BIT_2: ADDER_74LS283N.14, REGISTER_1_SN74LS273.6
- removed net REGISTER_1_OUT_BIT_3: ADDER_74LS283N.12, REGISTER_1_SN74LS273.9
- removed net REGISTER_2_OUT_BIT_0: ADDER_74LS283N.6, REGISTER_2_SN74LS273.2
- removed net REGISTER_2_OUT_BIT_1: ADDER_74LS283N.2, REGISTER_2_SN74LS273.5
- removed net REGISTER_2_OUT_BIT_2: ADDER_74LS283N.15, REGISTER_2_SN74LS273.6
- removed net REGISTER_2_OUT_BIT_3: ADDER_74LS283N.11, REGISTER_2_SN74LS273.9
- new net CTRL_OFF_1: CONTROLLER.1, CONTROLLER_INV_.13, REGISTER_1_CLEAR_CX.1
- new net CTRL_OFF_2: CONTROLLER.2, CONTROLLER_INV_.11, REGISTER_2_CLEAR_CX.1
- new net CTRL_OFF_3: CONTROLLER.3, CONTROLLER_INV_.9
- new net CTRL_OFF_4: CONTROLLER.4, CONTROLLER_INV_.1
- new net CTRL_OFF_5: CONTROLLER.5, CONTROLLER_INV_.3
- new net CTRL_OFF_6: CONTROLLER.6, CONTROLLER_INV_.5
- new net CTRL_ON_1: CONTROLLER_INV_.12
- new net CTRL_ON_2: CONTROLLER_INV_.10
- new net CTRL_ON_3: CONTROLLER_INV_.8
- new net CTRL_ON_4: CONTROLLER_INV_.2
- new net CTRL_ON_5: CONTROLLER_INV_.4
- new net CTRL_ON_6: CONTROLLER_INV_.6
- new net PC_0: CONTROLLER.15, PRG_COUNTER.1, PRG_COUNTER.12
- new net PC_1: CONTROLLER.14, PRG_COUNTER.9
- new net PC_2: CONTROLLER.13, PRG_COUNTER.8
- new net PC_3: CONTROLLER.12, PRG_COUNTER.11
- net DTA_BUS_0: now also DISPLAY_DRIVER.7; no longer DISPLAY_DRIVER_74LS47.7
- net DTA_BUS_1: now also DISPLAY_DRIVER.1; no longer DISPLAY_DRIVER_74LS47.1
- net DTA_BUS_2: now also DISPLAY_DRIVER.2; no longer DISPLAY_DRIVER_74LS47.2
- net DTA_BUS_3: now also DISPLAY_DRIVER.6; no longer DISPLAY_DRIVER_74LS47.6
- net GND: now also CONTROLLER.8, CONTROLLER_INV_.7, DISPLAY_DRIVER.8, PRG_COUNTER.10, PRG_COUNTER.2, PRG_COUNTER.3, PRG_COUNTER.6, PRG_COUNTER.7, REGISTER_1.10, REGISTER_1.13, REGISTER_1.14, REGISTER_1.17, REGISTER_1.18, REGISTER_2.10, REGISTER_2.13, REGISTER_2.14, REGISTER_2.17, REGISTER_2.18; no longer ADDER_74LS283N.7, ADDER_74LS283N.8, CONTROLLER_CD4017BE.13, CONTROLLER_CD4017BE.15, CONTROLLER_CD4017BE.8, CONTROLLER_INV_SN74LS14.7, DISPLAY_DRIVER_74LS47.8, REGISTER_1_SN74LS273.10, REGISTER_1_SN74LS273.13, REGISTER_1_SN74LS273.14, REGISTER_1_SN74LS273.17, REGISTER_1_SN74LS273.18, REGISTER_2_SN74LS273.10, REGISTER_2_SN74LS273.13, REGISTER_2_SN74LS273.14, REGISTER_2_SN74LS273.17, REGISTER_2_SN74LS273.18
- net REGISTER_1_CLK: now also REGISTER_1.11; no longer REGISTER_1_SN74LS273.11
- net REGISTER_1_CLR: now also REGISTER_1.1; no longer REGISTER_1_SN74LS273.1
- net REGISTER_1_IN_BIT_0: now also REGISTER_1.3; no longer REGISTER_1_SN74LS273.3
- net REGISTER_1_IN_BIT_1: now also REGISTER_1.4; no longer REGISTER_1_SN74LS273.4
- net REGISTER_1_IN_BIT_2: now also REGISTER_1.7; no longer REGISTER_1_SN74LS273.7
- net REGISTER_1_IN_BIT_3: now also REGISTER_1.8; no longer REGISTER_1_SN74LS273.8
- net REGISTER_2_CLK: now also REGISTER_2.11; no longer REGISTER_2_SN74LS273.11
- net REGISTER_2_CLR: now also REGISTER_2.1; no longer REGISTER_2_SN74LS273.1
- net REGISTER_2_IN_BIT_0: now also REGISTER_2.3; no longer REGISTER_2_SN74LS273.3
- net REGISTER_2_IN_BIT_1: now also REGISTER_2.4; no longer REGISTER_2_SN74LS273.4
- net REGISTER_2_IN_BIT_2: now also REGISTER_2.7; no longer REGISTER_2_SN74LS273.7
- net REGISTER_2_IN_BIT_3: now also REGISTER_2.8; no longer REGISTER_2_SN74LS273.8
- net SEG_1_DA: now also DISPLAY_DRIVER.13; no longer DISPLAY_DRIVER_74LS47.13
- net SEG_1_DB: now also DISPLAY_DRIVER.12; no longer DISPLAY_DRIVER_74LS47.12
- net SEG_1_DC: now also DISPLAY_DRIVER.11; no longer DISPLAY_DRIVER_74LS47.11
- net SEG_1_DD: now also DISPLAY_DRIVER.10; no longer DISPLAY_DRIVER_74LS47.10
- net SEG_1_DE: now also DISPLAY_DRIVER.9; no longer DISPLAY_DRIVER_74LS47.9
- net SEG_1_DF: now also DISPLAY_DRIVER.15; no longer DISPLAY_DRIVER_74LS47.15
- net SEG_1_DG: now also DISPLAY_DRIVER.14; no longer DISPLAY_DRIVER_74LS47.14
- net TMR555_OUTPUT: now also PRG_COUNTER.14; no longer CONTROLLER_CD4017BE.14
- net VCC: now also CONTROLLER.16, CONTROLLER_INV_.14, DISPLAY_DRIVER.16, DISPLAY_DRIVER.3, DISPLAY_DRIVER.4, DISPLAY_DRIVER.5, PRG_COUNTER.5, REGISTER_1.20, REGISTER_2.20; no longer ADDER_74LS283N.16, CONTROLLER_CD4017BE.16, CONTROLLER_INV_SN74LS14.14, DISPLAY_DRIVER_74LS47.16, DISPLAY_DRIVER_74LS47.3, DISPLAY_DRIVER_74LS47.4, DISPLAY_DRIVER_74LS47.5, REGISTER_1_SN74LS273.20, REGISTER_2_SN74LS273.20
