File: EXTENSIONS/Analog/fCPU/v1.WithProgramCounterAndControllerAsSN74LS42N/fCPU.sch (EAGLE design)
At the start: 15 parts

Commit message: Update fCPU
Parts:
- removed ADDER_74LS283N: 74LS283N, 74xx-us:74LS283N
- removed CONTROLLER_CD4017BE: CD4017, SparkFun-DigitalIC:CD4017
- added CONTROLLER: 74LS42N, 74xx-us:74LS42N
- added PRG_COUNTER: 74LS90N, 74xx-us:74LS90N
- renumbered CONTROLLER_INV_SN74LS14 to CONTROLLER_INV_, DISPLAY_DRIVER_74LS47 to DISPLAY_DRIVER, REGISTER_1_SN74LS273 to REGISTER_1, REGISTER_2_SN74LS273 to REGISTER_2
Connections:
- net CTRL_LOW_3 renamed CTRL_ON_3
- net CTRL_LOW_4 renamed CTRL_ON_4
- net CTRL_LOW_5 renamed CTRL_ON_5
- net CTRL_LOW_6 renamed CTRL_ON_6
- removed net CTRL_HIGH_1: CONTROLLER_CD4017BEA.Q0, CONTROLLER_INV_A.I
- removed net CTRL_HIGH_2: CONTROLLER_CD4017BEA.Q1, CONTROLLER_INV_B.I
- removed net CTRL_HIGH_3: CONTROLLER_CD4017BEA.Q2, CONTROLLER_INV_C.I
- removed net CTRL_HIGH_4: CONTROLLER_CD4017BEA.Q3, CONTROLLER_INV_D.I
- removed net CTRL_HIGH_5: CONTROLLER_CD4017BEA.Q4, CONTROLLER_INV_E.I
- removed net CTRL_HIGH_6: CONTROLLER_CD4017BEA.Q5, CONTROLLER_INV_F.I
- removed net CTRL_LOW_1: CONTROLLER_INV_A.O, REGISTER_1_CLEAR_CX.1
- removed net CTRL_LOW_2: CONTROLLER_INV_B.O, REGISTER_2_CLEAR_CX.1
- removed net N$10: ADDER_74LS283NA.S1
- removed net N$11: ADDER_74LS283NA.S2
- removed net N$12: ADDER_74LS283NA.S3
- removed net N$13: ADDER_74LS283NA.S4
- removed net REGISTER_1_OUT_BIT_0: ADDER_74LS283NA.A1, REGISTER_1A.Q1
- removed net REGISTER_1_OUT_BIT_1: ADDER_74LS283NA.A2, REGISTER_1A.Q2
- removed net REGISTER_1_OUT_BIT_2: ADDER_74LS283NA.A3, REGISTER_1A.Q3
- removed net REGISTER_1_OUT_BIT_3: ADDER_74LS283NA.A4, REGISTER_1A.Q4
- removed net REGISTER_2_OUT_BIT_0: ADDER_74LS283NA.B1, REGISTER_2A.Q1
- removed net REGISTER_2_OUT_BIT_1: ADDER_74LS283NA.B2, REGISTER_2A.Q2
- removed net REGISTER_2_OUT_BIT_2: ADDER_74LS283NA.B3, REGISTER_2A.Q3
- removed net REGISTER_2_OUT_BIT_3: ADDER_74LS283NA.B4, REGISTER_2A.Q4
- new net CTRL_OFF_1: CONTROLLERA.O0, CONTROLLER_INV_A.I, REGISTER_1_CLEAR_CX.1
- new net CTRL_OFF_2: CONTROLLERA.O1, CONTROLLER_INV_B.I, REGISTER_2_CLEAR_CX.1
- new net CTRL_OFF_3: CONTROLLERA.O2, CONTROLLER_INV_C.I
- new net CTRL_OFF_4: CONTROLLERA.O3, CONTROLLER_INV_D.I
- new net CTRL_OFF_5: CONTROLLERA.O4, CONTROLLER_INV_E.I
- new net CTRL_OFF_6: CONTROLLERA.O5, CONTROLLER_INV_F.I
- new net CTRL_ON_1: CONTROLLER_INV_A.O
- new net CTRL_ON_2: CONTROLLER_INV_B.O
- new net PC_0: CONTROLLERA.A, PRG_COUNTERA.CKB, PRG_COUNTERA.QA
- new net PC_1: CONTROLLERA.B, PRG_COUNTERA.QB
- new net PC_2: CONTROLLERA.C, PRG_COUNTERA.QC
- new net PC_3: CONTROLLERA.D, PRG_COUNTERA.QD
- net GND: now also PRG_COUNTERA.R0(1), PRG_COUNTERA.R0(2), PRG_COUNTERA.R9(1), PRG_COUNTERA.R9(2); no longer ADDER_74LS283NA.C0, CONTROLLER_CD4017BEA.ENA, CONTROLLER_CD4017BEA.RES
- net TMR555_OUTPUT: now also PRG_COUNTERA.CKA; no longer CONTROLLER_CD4017BEA.CLK
