File: EXTENSIONS/Analog/fCPU/v1.WithCD4017NAsController/fCPU.sch (EAGLE design)
At the start: 17 parts

Commit message: Update fCPU
Parts:
- removed CLEAR_REGISTER_1, CLEAR_REGISTER_2, CLOCK_REGISTER_1, CLOCK_REGISTER_2: (no value), switch-omron:10-XX
- removed LED_POWER: (no value), adafruit:LEDSMT1206
- removed RESISTOR_SWITCHES: (no value), resistor-sip:4610X
- added CONTROLLER_CD4017BE: CD4017, SparkFun-DigitalIC:CD4017
- added CONTROLLER_INV_SN74LS14: 74LS14N, 74xx-us:74LS14N
- added REGISTER_1_CLEAR_CX, REGISTER_2_CLEAR_CX: (no value), microbuilder:SOLDERJUMPERREFLOW
Connections:
- removed net CLEAR_REGISTER_1_TO_GND: CLEAR_REGISTER_1.S, RESISTOR_SWITCHES.4
- removed net CLEAR_REGISTER_2_TO_GND: CLEAR_REGISTER_2.S, RESISTOR_SWITCHES.5
- removed net LED_POWER_TO_GND: LED_POWER.C, RESISTOR_SWITCHES.9
- new net CTRL_HIGH_1: CONTROLLER_CD4017BEA.Q0, CONTROLLER_INV_SN74LS14A.I
- new net CTRL_HIGH_2: CONTROLLER_CD4017BEA.Q1, CONTROLLER_INV_SN74LS14B.I
- new net CTRL_HIGH_3: CONTROLLER_CD4017BEA.Q2, CONTROLLER_INV_SN74LS14C.I
- new net CTRL_HIGH_4: CONTROLLER_CD4017BEA.Q3, CONTROLLER_INV_SN74LS14D.I
- new net CTRL_HIGH_5: CONTROLLER_CD4017BEA.Q4, CONTROLLER_INV_SN74LS14E.I
- new net CTRL_HIGH_6: CONTROLLER_CD4017BEA.Q5, CONTROLLER_INV_SN74LS14F.I
- new net CTRL_LOW_1: CONTROLLER_INV_SN74LS14A.O, REGISTER_1_CLEAR_CX.1
- new net CTRL_LOW_2: CONTROLLER_INV_SN74LS14B.O, REGISTER_2_CLEAR_CX.1
- new net CTRL_LOW_3: CONTROLLER_INV_SN74LS14C.O
- new net CTRL_LOW_4: CONTROLLER_INV_SN74LS14D.O
- new net CTRL_LOW_5: CONTROLLER_INV_SN74LS14E.O
- new net CTRL_LOW_6: CONTROLLER_INV_SN74LS14F.O
- new net N$10: ADDER_74LS283NA.S1
- new net N$11: ADDER_74LS283NA.S2
- new net N$12: ADDER_74LS283NA.S3
- new net N$13: ADDER_74LS283NA.S4
- net DTA_BUS_0: no longer ADDER_74LS283NA.S1
- net DTA_BUS_1: no longer ADDER_74LS283NA.S2
- net DTA_BUS_2: no longer ADDER_74LS283NA.S3
- net DTA_BUS_3: no longer ADDER_74LS283NA.S4
- net GND: now also CONTROLLER_CD4017BEA.ENA, CONTROLLER_CD4017BEA.RES; no longer RESISTOR_SWITCHES.1
- net REGISTER_1_CLK: no longer CLOCK_REGISTER_1.P1, RESISTOR_SWITCHES.2
- net REGISTER_1_CLR: now also REGISTER_1_CLEAR_CX.2; no longer CLEAR_REGISTER_1.P1
- net REGISTER_2_CLK: no longer CLOCK_REGISTER_2.P1, RESISTOR_SWITCHES.3
- net REGISTER_2_CLR: now also REGISTER_2_CLEAR_CX.2; no longer CLEAR_REGISTER_2.P1
- net TMR555_OUTPUT: now also CONTROLLER_CD4017BEA.CLK
- net VCC: no longer CLOCK_REGISTER_1.S, CLOCK_REGISTER_2.S, LED_POWER.A
