File: EXTENSIONS/Analog/fCPU/fCPU.sch (EAGLE design)
At the start: 15 parts

Commit message: Update fCPU
Parts:
- removed CONTROLLER_CD4017BE: CD4017, SparkFun-DigitalIC:CD4017
- removed CONTROLLER_INV_SN74LS14: 74LS14N, 74xx-us:74LS14N
- removed REGISTER_1_CLEAR_CX, REGISTER_2_CLEAR_CX: (no value), microbuilder:SOLDERJUMPERREFLOW
- added CLEAR_REGISTER_1, CLEAR_REGISTER_2, CLOCK_REGISTER_1, CLOCK_REGISTER_2: (no value), switch-omron:10-XX
- added LED_POWER: (no value), adafruit:LEDSMT1206
- added RESISTOR_SWITCHES: (no value), resistor-sip:4610X
Connections:
- removed net CTRL_HIGH_1: CONTROLLER_CD4017BEA.Q0, CONTROLLER_INV_SN74LS14A.I
- removed net CTRL_HIGH_2: CONTROLLER_CD4017BEA.Q1, CONTROLLER_INV_SN74LS14B.I
- removed net CTRL_HIGH_3: CONTROLLER_CD4017BEA.Q2, CONTROLLER_INV_SN74LS14C.I
- removed net CTRL_HIGH_4: CONTROLLER_CD4017BEA.Q3, CONTROLLER_INV_SN74LS14D.I
- removed net CTRL_HIGH_5: CONTROLLER_CD4017BEA.Q4, CONTROLLER_INV_SN74LS14E.I
- removed net CTRL_HIGH_6: CONTROLLER_CD4017BEA.Q5, CONTROLLER_INV_SN74LS14F.I
- removed net CTRL_LOW_1: CONTROLLER_INV_SN74LS14A.O, REGISTER_1_CLEAR_CX.1
- removed net CTRL_LOW_2: CONTROLLER_INV_SN74LS14B.O, REGISTER_2_CLEAR_CX.1
- removed net CTRL_LOW_3: CONTROLLER_INV_SN74LS14C.O
- removed net CTRL_LOW_4: CONTROLLER_INV_SN74LS14D.O
- removed net CTRL_LOW_5: CONTROLLER_INV_SN74LS14E.O
- removed net CTRL_LOW_6: CONTROLLER_INV_SN74LS14F.O
- removed net N$10: ADDER_74LS283NA.S1
- removed net N$11: ADDER_74LS283NA.S2
- removed net N$12: ADDER_74LS283NA.S3
- removed net N$13: ADDER_74LS283NA.S4
- new net CLEAR_REGISTER_1_TO_GND: CLEAR_REGISTER_1.S, RESISTOR_SWITCHES.4
- new net CLEAR_REGISTER_2_TO_GND: CLEAR_REGISTER_2.S, RESISTOR_SWITCHES.5
- new net LED_POWER_TO_GND: LED_POWER.C, RESISTOR_SWITCHES.9
- net DTA_BUS_0: now also ADDER_74LS283NA.S1
- net DTA_BUS_1: now also ADDER_74LS283NA.S2
- net DTA_BUS_2: now also ADDER_74LS283NA.S3
- net DTA_BUS_3: now also ADDER_74LS283NA.S4
- net GND: now also RESISTOR_SWITCHES.1; no longer CONTROLLER_CD4017BEA.ENA, CONTROLLER_CD4017BEA.RES
- net REGISTER_1_CLK: now also CLOCK_REGISTER_1.P1, RESISTOR_SWITCHES.2
- net REGISTER_1_CLR: now also CLEAR_REGISTER_1.P1; no longer REGISTER_1_CLEAR_CX.2
- net REGISTER_2_CLK: now also CLOCK_REGISTER_2.P1, RESISTOR_SWITCHES.3
- net REGISTER_2_CLR: now also CLEAR_REGISTER_2.P1; no longer REGISTER_2_CLEAR_CX.2
- net TMR555_OUTPUT: no longer CONTROLLER_CD4017BEA.CLK
- net VCC: now also CLOCK_REGISTER_1.S, CLOCK_REGISTER_2.S, LED_POWER.A

Commit message: Update fCPU
Connections:
- net TMR555_OUTPUT: now also LED_POWER.A
- net VCC: no longer LED_POWER.A
Changed lines of the file:
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@@
 <label x="-27.94" y="213.36" size="1.778" layer="95"/>
-</segment>
-<segment>
-<pinref part="LED_POWER" gate="G$1" pin="A"/>
-<wire x1="78.74" y1="195.58" x2="78.74" y2="205.74" width="0.1524" layer="91"/>
-<label x="78.74" y="203.2" size="1.778" layer="95"/>
 </segment>
 </net>
@@
 <label x="33.02" y="104.14" size="1.778" layer="95"/>
 </segment>
+<segment>
+<pinref part="LED_POWER" gate="G$1" pin="A"/>
+<wire x1="78.74" y1="195.58" x2="78.74" y2="205.74" width="0.1524" layer="91"/>
+<label x="78.74" y="203.2" size="1.778" layer="95"/>
+</segment>
 </net>

Commit message: Update fCPU
Parts:
- added INPUT_DEVICE_1_EX, INPUT_DEVICE_2_EX: (no value), pinhead:PINHD-1X4
Connections:
- net REGISTER_1_IN_BIT_0: now also INPUT_DEVICE_1_EX.1
- net REGISTER_1_IN_BIT_1: now also INPUT_DEVICE_1_EX.2
- net REGISTER_1_IN_BIT_2: now also INPUT_DEVICE_1_EX.3
- net REGISTER_1_IN_BIT_3: now also INPUT_DEVICE_1_EX.4
- net REGISTER_2_IN_BIT_0: now also INPUT_DEVICE_2_EX.1
- net REGISTER_2_IN_BIT_1: now also INPUT_DEVICE_2_EX.2
- net REGISTER_2_IN_BIT_2: now also INPUT_DEVICE_2_EX.3
- net REGISTER_2_IN_BIT_3: now also INPUT_DEVICE_2_EX.4
Changed lines of the file:
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@@
 <part name="CLEAR_REGISTER_2" library="switch-omron" deviceset="10-XX" device=""/>
 <part name="LED_POWER" library="adafruit" deviceset="LED" device="SMT1206"/>
+<part name="INPUT_DEVICE_1_EX" library="pinhead" deviceset="PINHD-1X4" device=""/>
+<part name="INPUT_DEVICE_2_EX" library="pinhead" deviceset="PINHD-1X4" device=""/>
 </parts>
 <sheets>
@@
 <instance part="CLEAR_REGISTER_2" gate="1" x="-45.72" y="132.08"/>
 <instance part="LED_POWER" gate="G$1" x="78.74" y="193.04"/>
+<instance part="INPUT_DEVICE_1_EX" gate="A" x="289.56" y="152.4" smashed="yes" rot="R180">
+<attribute name="NAME" x="306.07" y="144.145" size="1.778" layer="95" rot="R180"/>
+<attribute name="VALUE" x="295.91" y="160.02" size="1.778" layer="96" rot="R180"/>
+</instance>
+<instance part="INPUT_DEVICE_2_EX" gate="A" x="289.56" y="132.08" smashed="yes" rot="R180">
+<attribute name="NAME" x="306.07" y="123.825" size="1.778" layer="95" rot="R180"/>
+<attribute name="VALUE" x="295.91" y="139.7" size="1.778" layer="96" rot="R180"/>
+</instance>
 </instances>
 <busses>
@@
 <pinref part="CLOCK_REGISTER_1" gate="1" pin="P1"/>
 <wire x1="-5.08" y1="190.5" x2="-5.08" y2="172.72" width="0.1524" layer="91"/>
-<label x="-7.62" y="170.18" size="1.778" layer="95"/>
+<label x="-10.16" y="175.26" size="1.778" layer="95"/>
 </segment>
 <segment>
@@
 <pinref part="CLOCK_REGISTER_2" gate="1" pin="P1"/>
 <wire x1="-25.4" y1="190.5" x2="-25.4" y2="175.26" width="0.1524" layer="91"/>
-<label x="-35.56" y="170.18" size="1.778" layer="95"/>
+<label x="-33.782" y="175.514" size="1.778" layer="95"/>
 </segment>
 <segment>
@@
 <label x="209.296" y="89.916" size="1.778" layer="95" rot="R270"/>
 </segment>
+<segment>
+<pinref part="INPUT_DEVICE_1_EX" gate="A" pin="1"/>
+<wire x1="292.1" y1="147.32" x2="309.88" y2="147.32" width="0.1524" layer="91"/>
+<label x="321.564" y="148.844" size="1.778" layer="95" rot="R180"/>
+</segment>
 </net>
 <net name="REGISTER_1_IN_BIT_1" class="0">
@@
 <label x="213.868" y="65.532" size="1.778" layer="95" rot="R90"/>
 </segment>
+<segment>
+<pinref part="INPUT_DEVICE_1_EX" gate="A" pin="2"/>
+<wire x1="292.1" y1="149.86" x2="309.88" y2="149.86" width="0.1524" layer="91"/>
+<label x="322.326" y="151.638" size="1.778" layer="95" rot="R180"/>
+</segment>
 </net>
 <net name="REGISTER_1_IN_BIT_2" class="0">
@@
 <label x="216.408" y="65.786" size="1.778" layer="95" rot="R90"/>
 </segment>
+<segment>
+<pinref part="INPUT_DEVICE_1_EX" gate="A" pin="3"/>
+<wire x1="292.1" y1="152.4" x2="307.34" y2="152.4" width="0.1524" layer="91"/>
+<label x="321.564" y="154.178" size="1.778" layer="95" rot="R180"/>
+</segment>
 </net>
 <net name="REGISTER_1_IN_BIT_3" class="0">
@@
 <label x="219.202" y="65.786" size="1.778" layer="95" rot="R90"/>
 </segment>
+<segment>
+<pinref part="INPUT_DEVICE_1_EX" gate="A" pin="4"/>
+<wire x1="292.1" y1="154.94" x2="317.5" y2="154.94" width="0.1524" layer="91"/>
+<label x="321.818" y="157.988" size="1.778" layer="95" rot="R180"/>
+</segment>
 </net>
 <net name="REGISTER_2_IN_BIT_0" class="0">
@@
 <label x="221.996" y="62.23" size="1.778" layer="95" rot="R90"/>
 </segment>
+<segment>
+<pinref part="INPUT_DEVICE_2_EX" gate="A" pin="1"/>
+<wire x1="292.1" y1="127" x2="314.96" y2="127" width="0.1524" layer="91"/>
+<label x="312.42" y="127" size="1.778" layer="95"/>
+</segment>
 </net>
 <net name="REGISTER_2_IN_BIT_1" class="0">
@@
 <label x="224.536" y="61.976" size="1.778" layer="95" rot="R90"/>
 </segment>
+<segment>
+<pinref part="INPUT_DEVICE_2_EX" gate="A" pin="2"/>
+<wire x1="292.1" y1="129.54" x2="314.96" y2="129.54" width="0.1524" layer="91"/>
+<label x="312.42" y="129.54" size="1.778" layer="95"/>
+</segment>
 </net>
 <net name="REGISTER_2_IN_BIT_2" class="0">
@@
 <label x="227.33" y="61.976" size="1.778" layer="95" rot="R90"/>
 </segment>
+<segment>
+<pinref part="INPUT_DEVICE_2_EX" gate="A" pin="3"/>
+<wire x1="292.1" y1="132.08" x2="314.96" y2="132.08" width="0.1524" layer="91"/>
+<label x="312.42" y="132.08" size="1.778" layer="95"/>
+</segment>
 </net>
 <net name="REGISTER_2_IN_BIT_3" class="0">
@@
 <label x="231.14" y="61.976" size="1.778" layer="95" rot="R90"/>
 </segment>
-</net>
+<segment>
+<pinref part="INPUT_DEVICE_2_EX" gate="A" pin="4"/>
+<wire x1="292.1" y1="134.62" x2="314.96" y2="134.62" width="0.1524" layer="91"/>
+<label x="312.42" y="134.62" size="1.778" layer="95"/>
+</segment>
+</net>
