File: EXTENSIONS/Analog/fCPU/bu/fCPU.brd (EAGLE design)
At the start: 88 x 71 mm, 7 parts, among them IC1 74LS42N

Commit message: Create fCPU
Parts:
- removed IC1: 74LS42N, 74xx-us:DIL16
- removed SN74LS90N_0: 74LS90N, 74xx-us:DIL14
- added CONTROLLER: 74LS42N, 74xx-us:DIL16
- added CONTROLLER_INV_: 74LS14N, 74xx-us:DIL14
- added PRG_COUNTER: 74LS90N, 74xx-us:DIL14
- added REGISTER_1: 74273N, 74xx-us:DIL20
- added REG_1_BIT_0_DIODE, REG_1_BIT_1_DIODE, REG_1_BIT_2_DIODE, REG_1_BIT_3_DIODE: (no value), diode:MELF-MLL41
- renumbered 74LS47N_0 to DISPLAY_DRIVER
Connections:
- removed net CTRL_1: IC1.1
- removed net CTRL_2: IC1.2
- removed net CTRL_3: IC1.3
- removed net CTRL_4: IC1.4
- removed net CTRL_5: IC1.5
- removed net CTRL_6: IC1.6
- removed net DISPLAY_0: DISPLAY_DRIVER.7
- removed net DISPLAY_1: DISPLAY_DRIVER.1
- removed net DISPLAY_2: DISPLAY_DRIVER.2
- removed net DISPLAY_3: DISPLAY_DRIVER.6
- new net CTRL_ON_1: CONTROLLER.1, CONTROLLER_INV_.13
- new net CTRL_ON_2: CONTROLLER.2, CONTROLLER_INV_.11
- new net CTRL_ON_3: CONTROLLER.3, CONTROLLER_INV_.9
- new net CTRL_ON_4: CONTROLLER.4, CONTROLLER_INV_.1
- new net CTRL_ON_5: CONTROLLER.5, CONTROLLER_INV_.3
- new net CTRL_ON_6: CONTROLLER.6, CONTROLLER_INV_.5
- new net CTRL_ON_INV_1: CONTROLLER_INV_.12
- new net CTRL_ON_INV_2: CONTROLLER_INV_.10
- new net CTRL_ON_INV_3: CONTROLLER_INV_.8
- new net CTRL_ON_INV_4: CONTROLLER_INV_.2
- new net CTRL_ON_INV_5: CONTROLLER_INV_.4
- new net CTRL_ON_INV_6: CONTROLLER_INV_.6
- new net DTA_BUS_0: DISPLAY_DRIVER.7, REG_1_BIT_0_DIODE.C
- new net DTA_BUS_1: DISPLAY_DRIVER.1, REG_1_BIT_1_DIODE.C
- new net DTA_BUS_2: DISPLAY_DRIVER.2, REG_1_BIT_2_DIODE.C
- new net DTA_BUS_3: DISPLAY_DRIVER.6, REG_1_BIT_3_DIODE.C
- new net N$2: REGISTER_1.2, REG_1_BIT_0_DIODE.A
- new net N$3: REGISTER_1.5, REG_1_BIT_1_DIODE.A
- new net N$4: REGISTER_1.6, REG_1_BIT_2_DIODE.A
- new net N$5: REGISTER_1.9, REG_1_BIT_3_DIODE.A
- new net REGISTER_1_CLK: REGISTER_1.11
- new net REGISTER_1_CLR: REGISTER_1.1
- net GND: now also CONTROLLER.8, CONTROLLER_INV_.7, PRG_COUNTER.10, PRG_COUNTER.2, PRG_COUNTER.3, PRG_COUNTER.6, PRG_COUNTER.7, REGISTER_1.10; no longer IC1.8, SN74LS90N_0.10, SN74LS90N_0.2, SN74LS90N_0.3, SN74LS90N_0.6, SN74LS90N_0.7
- net PC_0: now also CONTROLLER.15, PRG_COUNTER.1, PRG_COUNTER.12; no longer IC1.15, SN74LS90N_0.1, SN74LS90N_0.12
- net PC_1: now also CONTROLLER.14, PRG_COUNTER.9; no longer IC1.14, SN74LS90N_0.9
- net PC_2: now also CONTROLLER.13, PRG_COUNTER.8; no longer IC1.13, SN74LS90N_0.8
- net PC_3: now also CONTROLLER.12, PRG_COUNTER.11; no longer IC1.12, SN74LS90N_0.11
- net TMR555_OUTPUT: now also PRG_COUNTER.14; no longer SN74LS90N_0.14
- net VCC: now also CONTROLLER.16, CONTROLLER_INV_.14, PRG_COUNTER.5, REGISTER_1.20; no longer IC1.16, SN74LS90N_0.5

Commit message: Create fCPU
Parts:
- added REGISTER_1_CLEAR_CX: (no value), microbuilder:SOLDERJUMPER_REFLOW
Connections:
- removed net CTRL_ON_INV_1: CONTROLLER_INV_.12
- removed net CTRL_ON_INV_2: CONTROLLER_INV_.10
- removed net CTRL_ON_INV_3: CONTROLLER_INV_.8
- removed net CTRL_ON_INV_4: CONTROLLER_INV_.2
- removed net CTRL_ON_INV_5: CONTROLLER_INV_.4
- removed net CTRL_ON_INV_6: CONTROLLER_INV_.6
- new net CTRL_OFF_1: CONTROLLER.1, CONTROLLER_INV_.13, REGISTER_1_CLEAR_CX.1
- new net CTRL_OFF_2: CONTROLLER.2, CONTROLLER_INV_.11
- new net CTRL_OFF_3: CONTROLLER.3, CONTROLLER_INV_.9
- new net CTRL_OFF_4: CONTROLLER.4, CONTROLLER_INV_.1
- new net CTRL_OFF_5: CONTROLLER.5, CONTROLLER_INV_.3
- new net CTRL_OFF_6: CONTROLLER.6, CONTROLLER_INV_.5
- net CTRL_ON_1: now also CONTROLLER_INV_.12; no longer CONTROLLER.1, CONTROLLER_INV_.13
- net CTRL_ON_2: now also CONTROLLER_INV_.10; no longer CONTROLLER.2, CONTROLLER_INV_.11
- net CTRL_ON_3: now also CONTROLLER_INV_.8; no longer CONTROLLER.3, CONTROLLER_INV_.9
- net CTRL_ON_4: now also CONTROLLER_INV_.2; no longer CONTROLLER.4, CONTROLLER_INV_.1
- net CTRL_ON_5: now also CONTROLLER_INV_.4; no longer CONTROLLER.5, CONTROLLER_INV_.3
- net CTRL_ON_6: now also CONTROLLER_INV_.6; no longer CONTROLLER.6, CONTROLLER_INV_.5
- net REGISTER_1_CLR: now also REGISTER_1_CLEAR_CX.2
Changed lines of the file:
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@@
 <element name="REG_1_BIT_1_DIODE" library="diode" package="MELF-MLL41" value="" x="78" y="22" rot="R180"/>
 <element name="REG_1_BIT_0_DIODE" library="diode" package="MELF-MLL41" value="" x="78" y="16" rot="R180"/>
+<element name="REGISTER_1_CLEAR_CX" library="microbuilder" package="SOLDERJUMPER_REFLOW" value="" x="47" y="51"/>
 </elements>
 <signals>
@@
 <wire x1="25.19" y1="65.69" x2="79.625" y2="32" width="0" layer="19" extent="1-1"/>
 </signal>
-<signal name="CTRL_ON_1">
-<contactref element="CONTROLLER" pad="1"/>
-<contactref element="CONTROLLER_INV_" pad="13"/>
-<wire x1="19.19" y1="43.89" x2="39.81" y2="40.08" width="0" layer="19" extent="1-1"/>
+<signal name="CTRL_ON_3">
+<contactref element="CONTROLLER_INV_" pad="8"/>
 </signal>
 <signal name="CTRL_ON_2">
-<contactref element="CONTROLLER" pad="2"/>
-<contactref element="CONTROLLER_INV_" pad="11"/>
-<wire x1="19.19" y1="41.35" x2="39.81" y2="35" width="0" layer="19" extent="1-1"/>
-</signal>
-<signal name="CTRL_ON_3">
-<contactref element="CONTROLLER" pad="3"/>
-<contactref element="CONTROLLER_INV_" pad="9"/>
-<wire x1="19.19" y1="38.81" x2="39.81" y2="29.92" width="0" layer="19" extent="1-1"/>
+<contactref element="CONTROLLER_INV_" pad="10"/>
+</signal>
+<signal name="CTRL_ON_6">
+<contactref element="CONTROLLER_INV_" pad="6"/>
+</signal>
+<signal name="CTRL_ON_5">
+<contactref element="CONTROLLER_INV_" pad="4"/>
 </signal>
 <signal name="CTRL_ON_4">
-<contactref element="CONTROLLER" pad="4"/>
-<contactref element="CONTROLLER_INV_" pad="1"/>
-<wire x1="19.19" y1="36.27" x2="32.19" y2="42.62" width="0" layer="19" extent="1-1"/>
-</signal>
-<signal name="CTRL_ON_5">
-<contactref element="CONTROLLER" pad="5"/>
-<contactref element="CONTROLLER_INV_" pad="3"/>
-<wire x1="19.19" y1="33.73" x2="32.19" y2="37.54" width="0" layer="19" extent="1-1"/>
-</signal>
-<signal name="CTRL_ON_6">
-<contactref element="CONTROLLER" pad="6"/>
-<contactref element="CONTROLLER_INV_" pad="5"/>
-<wire x1="19.19" y1="31.19" x2="32.19" y2="32.46" width="0" layer="19" extent="1-1"/>
-</signal>
-<signal name="CTRL_ON_INV_3">
-<contactref element="CONTROLLER_INV_" pad="8"/>
-</signal>
-<signal name="CTRL_ON_INV_2">
-<contactref element="CONTROLLER_INV_" pad="10"/>
-</signal>
-<signal name="CTRL_ON_INV_1">
-<contactref element="CONTROLLER_INV_" pad="12"/>
-</signal>
-<signal name="CTRL_ON_INV_6">
-<contactref element="CONTROLLER_INV_" pad="6"/>
-</signal>
-<signal name="CTRL_ON_INV_5">
-<contactref element="CONTROLLER_INV_" pad="4"/>
-</signal>
-<signal name="CTRL_ON_INV_4">
 <contactref element="CONTROLLER_INV_" pad="2"/>
 </signal>
@@
 <signal name="REGISTER_1_CLR">
 <contactref element="REGISTER_1" pad="1"/>
+<contactref element="REGISTER_1_CLEAR_CX" pad="2"/>
+<wire x1="48.19" y1="38.43" x2="47.762" y2="51" width="0" layer="19" extent="1-1"/>
+</signal>
+<signal name="CTRL_OFF_1">
+<contactref element="CONTROLLER" pad="1"/>
+<contactref element="CONTROLLER_INV_" pad="13"/>
+<contactref element="REGISTER_1_CLEAR_CX" pad="1"/>
+<wire x1="39.81" y1="40.08" x2="46.238" y2="51" width="0" layer="19" extent="1-1"/>
+<wire x1="19.19" y1="43.89" x2="39.81" y2="40.08" width="0" layer="19" extent="1-1"/>
+</signal>
+<signal name="CTRL_OFF_2">
+<contactref element="CONTROLLER" pad="2"/>
+<contactref element="CONTROLLER_INV_" pad="11"/>
+<wire x1="19.19" y1="41.35" x2="39.81" y2="35" width="0" layer="19" extent="1-1"/>
+</signal>
+<signal name="CTRL_OFF_3">
+<contactref element="CONTROLLER" pad="3"/>
+<contactref element="CONTROLLER_INV_" pad="9"/>
+<wire x1="19.19" y1="38.81" x2="39.81" y2="29.92" width="0" layer="19" extent="1-1"/>
+</signal>
+<signal name="CTRL_OFF_4">
+<contactref element="CONTROLLER" pad="4"/>
+<contactref element="CONTROLLER_INV_" pad="1"/>
+<wire x1="19.19" y1="36.27" x2="32.19" y2="42.62" width="0" layer="19" extent="1-1"/>
+</signal>
+<signal name="CTRL_OFF_5">
+<contactref element="CONTROLLER" pad="5"/>
+<contactref element="CONTROLLER_INV_" pad="3"/>
+<wire x1="19.19" y1="33.73" x2="32.19" y2="37.54" width="0" layer="19" extent="1-1"/>
+</signal>
+<signal name="CTRL_OFF_6">
+<contactref element="CONTROLLER" pad="6"/>
+<contactref element="CONTROLLER_INV_" pad="5"/>
+<wire x1="19.19" y1="31.19" x2="32.19" y2="32.46" width="0" layer="19" extent="1-1"/>
+</signal>
+<signal name="CTRL_ON_1">
+<contactref element="CONTROLLER_INV_" pad="12"/>
 </signal>
 </signals>

Commit message: Update fCPU
Parts:
- removed REG_1_BIT_0_DIODE, REG_1_BIT_1_DIODE, REG_1_BIT_2_DIODE, REG_1_BIT_3_DIODE: (no value), diode:MELF-MLL41
- added INPUT_DEVICE_1, INPUT_DEVICE_2: (no value), special:EDG-04
- added REGISTER_2: 74273N, 74xx-us:DIL20
- added REGISTER_2_CLEAR_CX: (no value), microbuilder:SOLDERJUMPER_REFLOW
- added RESISTOR_INPUT_DEVICES: (no value), resistor-sip:SIP10
- moved CONTROLLER 19.8 mm to (9.00, 49.0)
- moved CONTROLLER_INV_ 15.6 mm to (24.0, 45.0)
- moved REGISTER_1_CLEAR_CX 12.2 mm to (35.0, 53.0)
- moved REGISTER_1 8.60 mm to (59.0, 32.0)
- moved PRG_COUNTER 8.06 mm to (9.00, 26.5)
Connections:
- removed net N$2: REGISTER_1.2, REG_1_BIT_0_DIODE.A
- removed net N$3: REGISTER_1.5, REG_1_BIT_1_DIODE.A
- removed net N$4: REGISTER_1.6, REG_1_BIT_2_DIODE.A
- removed net N$5: REGISTER_1.9, REG_1_BIT_3_DIODE.A
- new net REGISTER_1_IN_BIT_0: INPUT_DEVICE_1.1, REGISTER_1.3, RESISTOR_INPUT_DEVICES.2
- new net REGISTER_1_IN_BIT_1: INPUT_DEVICE_1.2, REGISTER_1.4, RESISTOR_INPUT_DEVICES.3
- new net REGISTER_1_IN_BIT_2: INPUT_DEVICE_1.3, REGISTER_1.7, RESISTOR_INPUT_DEVICES.4
- new net REGISTER_1_IN_BIT_3: INPUT_DEVICE_1.4, REGISTER_1.8, RESISTOR_INPUT_DEVICES.5
- new net REGISTER_2_CLK: REGISTER_2.11
- new net REGISTER_2_CLR: REGISTER_2.1, REGISTER_2_CLEAR_CX.2
- new net REGISTER_2_IN_BIT_0: INPUT_DEVICE_2.1, REGISTER_2.3, RESISTOR_INPUT_DEVICES.6
- new net REGISTER_2_IN_BIT_1: INPUT_DEVICE_2.2, REGISTER_2.4, RESISTOR_INPUT_DEVICES.7
- new net REGISTER_2_IN_BIT_2: INPUT_DEVICE_2.3, REGISTER_2.7, RESISTOR_INPUT_DEVICES.8
- new net REGISTER_2_IN_BIT_3: INPUT_DEVICE_2.4, REGISTER_2.8, RESISTOR_INPUT_DEVICES.9
- net CTRL_OFF_2: now also REGISTER_2_CLEAR_CX.1
- net DTA_BUS_0: no longer REG_1_BIT_0_DIODE.C
- net DTA_BUS_1: no longer REG_1_BIT_1_DIODE.C
- net DTA_BUS_2: no longer REG_1_BIT_2_DIODE.C
- net DTA_BUS_3: no longer REG_1_BIT_3_DIODE.C
- net GND: now also REGISTER_1.13, REGISTER_1.14, REGISTER_1.17, REGISTER_1.18, REGISTER_2.10, REGISTER_2.13, REGISTER_2.14, REGISTER_2.17, REGISTER_2.18, RESISTOR_INPUT_DEVICES.1
- net VCC: now also INPUT_DEVICE_1.5, INPUT_DEVICE_1.6, INPUT_DEVICE_1.7, INPUT_DEVICE_1.8, INPUT_DEVICE_2.5, INPUT_DEVICE_2.6, INPUT_DEVICE_2.7, INPUT_DEVICE_2.8, REGISTER_2.20
Other:
- board size 88 x 71 mm -> 97 x 73 mm

Commit message: Update fCPU
Parts:
- moved OUTPUTS 59.5 mm to (96.0, 19.5)
- moved JP_CLOCK_IN 29.5 mm to (49.5, 14.0)
- moved REGISTER_1 9.22 mm to (50.0, 34.0)
- moved REGISTER_2 9.22 mm to (50.0, 67.0)
- moved REGISTER_1_CLEAR_CX 8.25 mm to (43.0, 51.0)
- moved INPUT_DEVICE_1 2.24 mm to (86.0, 55.0)
Other:
- board text added: "PCBv1 - 2019.10"
- board text removed: "PCBv2 - 2019.09"
- board text removed: "https://bit.ly/2ZEPbGB"

Commit message: Update fCPU
Parts:
- removed CONTROLLER: 74LS42N, 74xx-us:DIL16
- removed CONTROLLER_INV_: 74LS14N, 74xx-us:DIL14
- removed DISPLAY_DRIVER: 74LS47N, 74xx-us:DIL16
- removed PRG_COUNTER: 74LS90N, 74xx-us:DIL14
- removed REGISTER_1, REGISTER_2: 74273N, 74xx-us:DIL20
- added ADDER_74LS283N: 74LS283N, 74xx-us:DIL16
- added CONTROLLER_CD4017BE: CD4017, SparkFun-DigitalIC:DIL16
- added CONTROLLER_INV_SN74LS14: 74LS14N, 74xx-us:DIL14
- added DISPLAY_DRIVER_74LS47: 74LS47N, 74xx-us:DIL16
- added REGISTER_1_SN74LS273, REGISTER_2_SN74LS273: 74273N, 74xx-us:DIL20
- moved DIGIT_0_ANODE 41.3 mm to (50.0, 67.0)
- moved R_100O_0 32.1 mm to (49.5, 80.5), turned to 180 degrees
- moved REGISTER_1_CLEAR_CX 19.3 mm to (50.0, 33.0)
- moved REGISTER_2_CLEAR_CX 12.0 mm to (48.0, 49.0)
Connections:
- removed net CTRL_OFF_1: CONTROLLER.1, CONTROLLER_INV_.13, REGISTER_1_CLEAR_CX.1
- removed net CTRL_OFF_2: CONTROLLER.2, CONTROLLER_INV_.11, REGISTER_2_CLEAR_CX.1
- removed net CTRL_OFF_3: CONTROLLER.3, CONTROLLER_INV_.9
- removed net CTRL_OFF_4: CONTROLLER.4, CONTROLLER_INV_.1
- removed net CTRL_OFF_5: CONTROLLER.5, CONTROLLER_INV_.3
- removed net CTRL_OFF_6: CONTROLLER.6, CONTROLLER_INV_.5
- removed net CTRL_ON_1: CONTROLLER_INV_.12
- removed net CTRL_ON_2: CONTROLLER_INV_.10
- removed net CTRL_ON_3: CONTROLLER_INV_.8
- removed net CTRL_ON_4: CONTROLLER_INV_.2
- removed net CTRL_ON_5: CONTROLLER_INV_.4
- removed net CTRL_ON_6: CONTROLLER_INV_.6
- removed net PC_0: CONTROLLER.15, PRG_COUNTER.1, PRG_COUNTER.12
- removed net PC_1: CONTROLLER.14, PRG_COUNTER.9
- removed net PC_2: CONTROLLER.13, PRG_COUNTER.8
- removed net PC_3: CONTROLLER.12, PRG_COUNTER.11
- new net CTRL_HIGH_1: CONTROLLER_CD4017BE.3, CONTROLLER_INV_SN74LS14.13
- new net CTRL_HIGH_2: CONTROLLER_CD4017BE.2, CONTROLLER_INV_SN74LS14.11
- new net CTRL_HIGH_3: CONTROLLER_CD4017BE.4, CONTROLLER_INV_SN74LS14.9
- new net CTRL_HIGH_4: CONTROLLER_CD4017BE.7, CONTROLLER_INV_SN74LS14.1
- new net CTRL_HIGH_5: CONTROLLER_CD4017BE.10, CONTROLLER_INV_SN74LS14.3
- new net CTRL_HIGH_6: CONTROLLER_CD4017BE.1, CONTROLLER_INV_SN74LS14.5
- new net CTRL_LOW_1: CONTROLLER_INV_SN74LS14.12, REGISTER_1_CLEAR_CX.1
- new net CTRL_LOW_2: CONTROLLER_INV_SN74LS14.10, REGISTER_2_CLEAR_CX.1
- new net CTRL_LOW_3: CONTROLLER_INV_SN74LS14.8
- new net CTRL_LOW_4: CONTROLLER_INV_SN74LS14.2
- new net CTRL_LOW_5: CONTROLLER_INV_SN74LS14.4
- new net CTRL_LOW_6: CONTROLLER_INV_SN74LS14.6
- new net N$10: ADDER_74LS283N.4
- new net N$11: ADDER_74LS283N.1
- new net N$12: ADDER_74LS283N.13
- new net N$13: ADDER_74LS283N.10
- new net REGISTER_1_OUT_BIT_0: ADDER_74LS283N.5, REGISTER_1_SN74LS273.2
- new net REGISTER_1_OUT_BIT_1: ADDER_74LS283N.3, REGISTER_1_SN74LS273.5
- new net REGISTER_1_OUT_BIT_2: ADDER_74LS283N.14, REGISTER_1_SN74LS273.6
- new net REGISTER_1_OUT_BIT_3: ADDER_74LS283N.12, REGISTER_1_SN74LS273.9
- new net REGISTER_2_OUT_BIT_0: ADDER_74LS283N.6, REGISTER_2_SN74LS273.2
- new net REGISTER_2_OUT_BIT_1: ADDER_74LS283N.2, REGISTER_2_SN74LS273.5
- new net REGISTER_2_OUT_BIT_2: ADDER_74LS283N.15, REGISTER_2_SN74LS273.6
- new net REGISTER_2_OUT_BIT_3: ADDER_74LS283N.11, REGISTER_2_SN74LS273.9
- net DTA_BUS_0: now also DISPLAY_DRIVER_74LS47.7; no longer DISPLAY_DRIVER.7
- net DTA_BUS_1: now also DISPLAY_DRIVER_74LS47.1; no longer DISPLAY_DRIVER.1
- net DTA_BUS_2: now also DISPLAY_DRIVER_74LS47.2; no longer DISPLAY_DRIVER.2
- net DTA_BUS_3: now also DISPLAY_DRIVER_74LS47.6; no longer DISPLAY_DRIVER.6
- net GND: now also ADDER_74LS283N.7, ADDER_74LS283N.8, CONTROLLER_CD4017BE.13, CONTROLLER_CD4017BE.15, CONTROLLER_CD4017BE.8, CONTROLLER_INV_SN74LS14.7, DISPLAY_DRIVER_74LS47.8, REGISTER_1_SN74LS273.10, REGISTER_1_SN74LS273.13, REGISTER_1_SN74LS273.14, REGISTER_1_SN74LS273.17, REGISTER_1_SN74LS273.18, REGISTER_2_SN74LS273.10, REGISTER_2_SN74LS273.13, REGISTER_2_SN74LS273.14, REGISTER_2_SN74LS273.17, REGISTER_2_SN74LS273.18; no longer CONTROLLER.8, CONTROLLER_INV_.7, DISPLAY_DRIVER.8, PRG_COUNTER.10, PRG_COUNTER.2, PRG_COUNTER.3, PRG_COUNTER.6, PRG_COUNTER.7, REGISTER_1.10, REGISTER_1.13, REGISTER_1.14, REGISTER_1.17, REGISTER_1.18, REGISTER_2.10, REGISTER_2.13, REGISTER_2.14, REGISTER_2.17, REGISTER_2.18
- net REGISTER_1_CLK: now also REGISTER_1_SN74LS273.11; no longer REGISTER_1.11
- net REGISTER_1_CLR: now also REGISTER_1_SN74LS273.1; no longer REGISTER_1.1
- net REGISTER_1_IN_BIT_0: now also REGISTER_1_SN74LS273.3; no longer REGISTER_1.3
- net REGISTER_1_IN_BIT_1: now also REGISTER_1_SN74LS273.4; no longer REGISTER_1.4
- net REGISTER_1_IN_BIT_2: now also REGISTER_1_SN74LS273.7; no longer REGISTER_1.7
- net REGISTER_1_IN_BIT_3: now also REGISTER_1_SN74LS273.8; no longer REGISTER_1.8
- net REGISTER_2_CLK: now also REGISTER_2_SN74LS273.11; no longer REGISTER_2.11
- net REGISTER_2_CLR: now also REGISTER_2_SN74LS273.1; no longer REGISTER_2.1
- net REGISTER_2_IN_BIT_0: now also REGISTER_2_SN74LS273.3; no longer REGISTER_2.3
- net REGISTER_2_IN_BIT_1: now also REGISTER_2_SN74LS273.4; no longer REGISTER_2.4
- net REGISTER_2_IN_BIT_2: now also REGISTER_2_SN74LS273.7; no longer REGISTER_2.7
- net REGISTER_2_IN_BIT_3: now also REGISTER_2_SN74LS273.8; no longer REGISTER_2.8
- net SEG_1_DA: now also DISPLAY_DRIVER_74LS47.13; no longer DISPLAY_DRIVER.13
- net SEG_1_DB: now also DISPLAY_DRIVER_74LS47.12; no longer DISPLAY_DRIVER.12
- net SEG_1_DC: now also DISPLAY_DRIVER_74LS47.11; no longer DISPLAY_DRIVER.11
- net SEG_1_DD: now also DISPLAY_DRIVER_74LS47.10; no longer DISPLAY_DRIVER.10
- net SEG_1_DE: now also DISPLAY_DRIVER_74LS47.9; no longer DISPLAY_DRIVER.9
- net SEG_1_DF: now also DISPLAY_DRIVER_74LS47.15; no longer DISPLAY_DRIVER.15
- net SEG_1_DG: now also DISPLAY_DRIVER_74LS47.14; no longer DISPLAY_DRIVER.14
- net TMR555_OUTPUT: now also CONTROLLER_CD4017BE.14; no longer PRG_COUNTER.14
- net VCC: now also ADDER_74LS283N.16, CONTROLLER_CD4017BE.16, CONTROLLER_INV_SN74LS14.14, DISPLAY_DRIVER_74LS47.16, DISPLAY_DRIVER_74LS47.3, DISPLAY_DRIVER_74LS47.4, DISPLAY_DRIVER_74LS47.5, REGISTER_1_SN74LS273.20, REGISTER_2_SN74LS273.20; no longer CONTROLLER.16, CONTROLLER_INV_.14, DISPLAY_DRIVER.16, DISPLAY_DRIVER.3, DISPLAY_DRIVER.4, DISPLAY_DRIVER.5, PRG_COUNTER.5, REGISTER_1.20, REGISTER_2.20

Commit message: Update fCPU
Parts:
- removed CONTROLLER_CD4017BE: CD4017, SparkFun-DigitalIC:DIL16
- removed CONTROLLER_INV_SN74LS14: 74LS14N, 74xx-us:DIL14
- removed REGISTER_1_CLEAR_CX, REGISTER_2_CLEAR_CX: (no value), microbuilder:SOLDERJUMPER_REFLOW
- added CLEAR_REGISTER_1, CLEAR_REGISTER_2, CLOCK_REGISTER_1, CLOCK_REGISTER_2: (no value), switch-omron:B3F-10XX
- added INPUT_DEVICE_1_EX, INPUT_DEVICE_2_EX: (no value), pinhead:1X04
- added LED_POWER: (no value), adafruit:1206
- added RESISTOR_SWITCHES: (no value), resistor-sip:SIP10
- moved ADDER_74LS283N 64.2 mm to (10.0, 70.0), turned to 270 degrees
- moved RESISTOR_INPUT_DEVICES 24.1 mm to (78.0, 78.0), turned to 180 degrees
- moved INPUT_DEVICE_1 20.1 mm to (84.0, 35.0)
- moved REGISTER_2_SN74LS273 12.6 mm to (54.5, 67.5)
- moved REGISTER_1_SN74LS273 12.4 mm to (54.0, 35.0)
- moved DISPLAY_DRIVER_74LS47 12.2 mm to (26.0, 69.5)
- moved DIGIT_0_ANODE 11.0 mm to (39.0, 66.0)
- moved R_100O_0 10.5 mm to (39.0, 79.5)
- moved INPUT_DEVICE_2 10.4 mm to (83.0, 58.0)
- moved OUTPUTS 1.58 mm to (96.5, 18.0)
Connections:
- removed net CTRL_HIGH_1: CONTROLLER_CD4017BE.3, CONTROLLER_INV_SN74LS14.13
- removed net CTRL_HIGH_2: CONTROLLER_CD4017BE.2, CONTROLLER_INV_SN74LS14.11
- removed net CTRL_HIGH_3: CONTROLLER_CD4017BE.4, CONTROLLER_INV_SN74LS14.9
- removed net CTRL_HIGH_4: CONTROLLER_CD4017BE.7, CONTROLLER_INV_SN74LS14.1
- removed net CTRL_HIGH_5: CONTROLLER_CD4017BE.10, CONTROLLER_INV_SN74LS14.3
- removed net CTRL_HIGH_6: CONTROLLER_CD4017BE.1, CONTROLLER_INV_SN74LS14.5
- removed net CTRL_LOW_1: CONTROLLER_INV_SN74LS14.12, REGISTER_1_CLEAR_CX.1
- removed net CTRL_LOW_2: CONTROLLER_INV_SN74LS14.10, REGISTER_2_CLEAR_CX.1
- removed net CTRL_LOW_3: CONTROLLER_INV_SN74LS14.8
- removed net CTRL_LOW_4: CONTROLLER_INV_SN74LS14.2
- removed net CTRL_LOW_5: CONTROLLER_INV_SN74LS14.4
- removed net CTRL_LOW_6: CONTROLLER_INV_SN74LS14.6
- removed net N$10: ADDER_74LS283N.4
- removed net N$11: ADDER_74LS283N.1
- removed net N$12: ADDER_74LS283N.13
- removed net N$13: ADDER_74LS283N.10
- new net CLEAR_REGISTER_1_TO_GND: CLEAR_REGISTER_1.1, RESISTOR_SWITCHES.4
- new net CLEAR_REGISTER_2_TO_GND: CLEAR_REGISTER_2.1, RESISTOR_SWITCHES.5
- new net LED_POWER_TO_GND: LED_POWER.C, RESISTOR_SWITCHES.9
- net DTA_BUS_0: now also ADDER_74LS283N.4
- net DTA_BUS_1: now also ADDER_74LS283N.1
- net DTA_BUS_2: now also ADDER_74LS283N.13
- net DTA_BUS_3: now also ADDER_74LS283N.10
- net GND: now also RESISTOR_SWITCHES.1; no longer CONTROLLER_CD4017BE.13, CONTROLLER_CD4017BE.15, CONTROLLER_CD4017BE.8, CONTROLLER_INV_SN74LS14.7
- net REGISTER_1_CLK: now also CLOCK_REGISTER_1.4, RESISTOR_SWITCHES.2
- net REGISTER_1_CLR: now also CLEAR_REGISTER_1.4; no longer REGISTER_1_CLEAR_CX.2
- net REGISTER_1_IN_BIT_0: now also INPUT_DEVICE_1_EX.1
- net REGISTER_1_IN_BIT_1: now also INPUT_DEVICE_1_EX.2
- net REGISTER_1_IN_BIT_2: now also INPUT_DEVICE_1_EX.3
- net REGISTER_1_IN_BIT_3: now also INPUT_DEVICE_1_EX.4
- net REGISTER_2_CLK: now also CLOCK_REGISTER_2.4, RESISTOR_SWITCHES.3
- net REGISTER_2_CLR: now also CLEAR_REGISTER_2.4; no longer REGISTER_2_CLEAR_CX.2
- net REGISTER_2_IN_BIT_0: now also INPUT_DEVICE_2_EX.1
- net REGISTER_2_IN_BIT_1: now also INPUT_DEVICE_2_EX.2
- net REGISTER_2_IN_BIT_2: now also INPUT_DEVICE_2_EX.3
- net REGISTER_2_IN_BIT_3: now also INPUT_DEVICE_2_EX.4
- net TMR555_OUTPUT: now also LED_POWER.A; no longer CONTROLLER_CD4017BE.14
- net VCC: now also CLOCK_REGISTER_1.1, CLOCK_REGISTER_2.1; no longer CONTROLLER_CD4017BE.16, CONTROLLER_INV_SN74LS14.14
Other:
- board size 97 x 73 mm -> 97 x 70 mm
- board text added: "+"
- board text added: "B0"
- board text added: "B1"
- board text added: "B2"
- board text added: "B3"
- board text added: "v 1"
