File: EXTENSIONS/Analog/fCPU/bu/fCPU.sch (EAGLE design)
At the start: 7 parts, among them IC1 74LS42N

Commit message: Create fCPU
Parts:
- added CONTROLLER_INV_: 74LS14N, 74xx-us:74LS14N
- added REGISTER_1: 74273N, 74xx-us:74273N
- added REG_1_BIT_0_DIODE, REG_1_BIT_1_DIODE, REG_1_BIT_2_DIODE, REG_1_BIT_3_DIODE: (no value), diode:DIODE-MELF-MLL41
- renumbered 74LS47N_0 to DISPLAY_DRIVER, IC1 to CONTROLLER, SN74LS90N_0 to PRG_COUNTER
Connections:
- removed net CTRL_1: CONTROLLERA.O0
- removed net CTRL_2: CONTROLLERA.O1
- removed net CTRL_3: CONTROLLERA.O2
- removed net CTRL_4: CONTROLLERA.O3
- removed net CTRL_5: CONTROLLERA.O4
- removed net CTRL_6: CONTROLLERA.O5
- removed net DISPLAY_0: DISPLAY_DRIVERG$1.IA
- removed net DISPLAY_1: DISPLAY_DRIVERG$1.IB
- removed net DISPLAY_2: DISPLAY_DRIVERG$1.IC
- removed net DISPLAY_3: DISPLAY_DRIVERG$1.ID
- new net CTRL_ON_1: CONTROLLERA.O0, CONTROLLER_INV_A.I
- new net CTRL_ON_2: CONTROLLERA.O1, CONTROLLER_INV_B.I
- new net CTRL_ON_3: CONTROLLERA.O2, CONTROLLER_INV_C.I
- new net CTRL_ON_4: CONTROLLERA.O3, CONTROLLER_INV_D.I
- new net CTRL_ON_5: CONTROLLERA.O4, CONTROLLER_INV_E.I
- new net CTRL_ON_6: CONTROLLERA.O5, CONTROLLER_INV_F.I
- new net CTRL_ON_INV_1: CONTROLLER_INV_A.O
- new net CTRL_ON_INV_2: CONTROLLER_INV_B.O
- new net CTRL_ON_INV_3: CONTROLLER_INV_C.O
- new net CTRL_ON_INV_4: CONTROLLER_INV_D.O
- new net CTRL_ON_INV_5: CONTROLLER_INV_E.O
- new net CTRL_ON_INV_6: CONTROLLER_INV_F.O
- new net DTA_BUS_0: DISPLAY_DRIVERG$1.IA, REG_1_BIT_0_DIODE.C
- new net DTA_BUS_1: DISPLAY_DRIVERG$1.IB, REG_1_BIT_1_DIODE.C
- new net DTA_BUS_2: DISPLAY_DRIVERG$1.IC, REG_1_BIT_2_DIODE.C
- new net DTA_BUS_3: DISPLAY_DRIVERG$1.ID, REG_1_BIT_3_DIODE.C
- new net N$2: REGISTER_1A.Q1, REG_1_BIT_0_DIODE.A
- new net N$3: REGISTER_1A.Q2, REG_1_BIT_1_DIODE.A
- new net N$4: REGISTER_1A.Q3, REG_1_BIT_2_DIODE.A
- new net N$5: REGISTER_1A.Q4, REG_1_BIT_3_DIODE.A
- new net REGISTER_1_CLK: REGISTER_1A.CLK
- new net REGISTER_1_CLR: REGISTER_1A.CLR

Commit message: Create fCPU
Parts:
- added REGISTER_1_CLEAR_CX: (no value), microbuilder:SOLDERJUMPERREFLOW
Connections:
- removed net CTRL_ON_INV_1: CONTROLLER_INV_A.O
- removed net CTRL_ON_INV_2: CONTROLLER_INV_B.O
- removed net CTRL_ON_INV_3: CONTROLLER_INV_C.O
- removed net CTRL_ON_INV_4: CONTROLLER_INV_D.O
- removed net CTRL_ON_INV_5: CONTROLLER_INV_E.O
- removed net CTRL_ON_INV_6: CONTROLLER_INV_F.O
- new net CTRL_OFF_1: CONTROLLERA.O0, CONTROLLER_INV_A.I, REGISTER_1_CLEAR_CX.1
- new net CTRL_OFF_2: CONTROLLERA.O1, CONTROLLER_INV_B.I
- new net CTRL_OFF_3: CONTROLLERA.O2, CONTROLLER_INV_C.I
- new net CTRL_OFF_4: CONTROLLERA.O3, CONTROLLER_INV_D.I
- new net CTRL_OFF_5: CONTROLLERA.O4, CONTROLLER_INV_E.I
- new net CTRL_OFF_6: CONTROLLERA.O5, CONTROLLER_INV_F.I
- net CTRL_ON_1: now also CONTROLLER_INV_A.O; no longer CONTROLLERA.O0, CONTROLLER_INV_A.I
- net CTRL_ON_2: now also CONTROLLER_INV_B.O; no longer CONTROLLERA.O1, CONTROLLER_INV_B.I
- net CTRL_ON_3: now also CONTROLLER_INV_C.O; no longer CONTROLLERA.O2, CONTROLLER_INV_C.I
- net CTRL_ON_4: now also CONTROLLER_INV_D.O; no longer CONTROLLERA.O3, CONTROLLER_INV_D.I
- net CTRL_ON_5: now also CONTROLLER_INV_E.O; no longer CONTROLLERA.O4, CONTROLLER_INV_E.I
- net CTRL_ON_6: now also CONTROLLER_INV_F.O; no longer CONTROLLERA.O5, CONTROLLER_INV_F.I
- net REGISTER_1_CLR: now also REGISTER_1_CLEAR_CX.2
Other:
- moved on the sheet: CONTROLLER_INV_D, CONTROLLER_INV_E, CONTROLLER_INV_F
Changed lines of the file:
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@@
 <part name="REG_1_BIT_1_DIODE" library="diode" deviceset="DIODE-" device="MELF-MLL41"/>
 <part name="REG_1_BIT_0_DIODE" library="diode" deviceset="DIODE-" device="MELF-MLL41"/>
+<part name="REGISTER_1_CLEAR_CX" library="microbuilder" deviceset="SOLDERJUMPER" device="REFLOW"/>
 </parts>
 <sheets>
@@
 <instance part="CONTROLLER_INV_" gate="B" x="-27.94" y="193.04"/>
 <instance part="CONTROLLER_INV_" gate="C" x="-27.94" y="208.28"/>
-<instance part="CONTROLLER_INV_" gate="D" x="35.56" y="177.8"/>
-<instance part="CONTROLLER_INV_" gate="E" x="35.56" y="190.5"/>
-<instance part="CONTROLLER_INV_" gate="F" x="33.02" y="205.74"/>
+<instance part="CONTROLLER_INV_" gate="D" x="43.18" y="177.8"/>
+<instance part="CONTROLLER_INV_" gate="E" x="43.18" y="190.5"/>
+<instance part="CONTROLLER_INV_" gate="F" x="40.64" y="205.74"/>
 <instance part="REGISTER_1" gate="A" x="111.76" y="142.24"/>
 <instance part="REG_1_BIT_3_DIODE" gate="G$1" x="132.08" y="147.32" smashed="yes">
@@
 <attribute name="VALUE" x="142.24" y="152.6286" size="1.778" layer="96"/>
 </instance>
+<instance part="REGISTER_1_CLEAR_CX" gate="1" x="119.38" y="99.06"/>
 </instances>
 <busses>
@@
 </segment>
 </net>
-<net name="CTRL_ON_1" class="0">
+<net name="CTRL_ON_3" class="0">
+<segment>
+<pinref part="CONTROLLER_INV_" gate="C" pin="O"/>
+<wire x1="-17.78" y1="208.28" x2="0" y2="208.28" width="0.1524" layer="91"/>
+<label x="-7.62" y="208.28" size="1.778" layer="95"/>
+</segment>
+</net>
+<net name="CTRL_ON_2" class="0">
+<segment>
+<pinref part="CONTROLLER_INV_" gate="B" pin="O"/>
+<wire x1="-17.78" y1="193.04" x2="0" y2="193.04" width="0.1524" layer="91"/>
+<label x="-7.62" y="193.04" size="1.778" layer="95"/>
+</segment>
+</net>
+<net name="CTRL_ON_6" class="0">
+<segment>
+<pinref part="CONTROLLER_INV_" gate="F" pin="O"/>
+<wire x1="50.8" y1="205.74" x2="63.5" y2="205.74" width="0.1524" layer="91"/>
+<label x="58.42" y="205.74" size="1.778" layer="95"/>
+</segment>
+</net>
+<net name="CTRL_ON_5" class="0">
+<segment>
+<pinref part="CONTROLLER_INV_" gate="E" pin="O"/>
+<wire x1="53.34" y1="190.5" x2="66.04" y2="190.5" width="0.1524" layer="91"/>
+<label x="66.04" y="190.5" size="1.778" layer="95"/>
+</segment>
+</net>
+<net name="CTRL_ON_4" class="0">
+<segment>
+<pinref part="CONTROLLER_INV_" gate="D" pin="O"/>
+<wire x1="53.34" y1="177.8" x2="66.04" y2="177.8" width="0.1524" layer="91"/>
+<label x="66.04" y="180.34" size="1.778" layer="95"/>
+</segment>
+</net>
+<net name="N$2" class="0">
+<segment>
+<pinref part="REG_1_BIT_0_DIODE" gate="G$1" pin="A"/>
+<pinref part="REGISTER_1" gate="A" pin="Q1"/>
+<wire x1="137.16" y1="154.94" x2="124.46" y2="154.94" width="0.1524" layer="91"/>
+</segment>
+</net>
+<net name="N$3" class="0">
+<segment>
+<pinref part="REG_1_BIT_1_DIODE" gate="G$1" pin="A"/>
+<pinref part="REGISTER_1" gate="A" pin="Q2"/>
+<wire x1="129.54" y1="152.4" x2="124.46" y2="152.4" width="0.1524" layer="91"/>
+</segment>
+</net>
+<net name="N$4" class="0">
+<segment>
+<pinref part="REG_1_BIT_2_DIODE" gate="G$1" pin="A"/>
+<pinref part="REGISTER_1" gate="A" pin="Q3"/>
+<wire x1="139.7" y1="149.86" x2="124.46" y2="149.86" width="0.1524" layer="91"/>
+</segment>
+</net>
+<net name="N$5" class="0">
+<segment>
+<pinref part="REG_1_BIT_3_DIODE" gate="G$1" pin="A"/>
+<pinref part="REGISTER_1" gate="A" pin="Q4"/>
+<wire x1="129.54" y1="147.32" x2="124.46" y2="147.32" width="0.1524" layer="91"/>
+</segment>
+</net>
+<net name="REGISTER_1_CLK" class="0">
+<segment>
+<pinref part="REGISTER_1" gate="A" pin="CLK"/>
+<wire x1="99.06" y1="132.08" x2="83.82" y2="132.08" width="0.1524" layer="91"/>
+<label x="78.74" y="132.08" size="1.778" layer="95"/>
+</segment>
+</net>
+<net name="REGISTER_1_CLR" class="0">
+<segment>
+<pinref part="REGISTER_1" gate="A" pin="CLR"/>
+<wire x1="99.06" y1="129.54" x2="73.66" y2="129.54" width="0.1524" layer="91"/>
+<label x="76.2" y="127" size="1.778" layer="95"/>
+</segment>
+<segment>
+<pinref part="REGISTER_1_CLEAR_CX" gate="1" pin="2"/>
+<wire x1="124.46" y1="99.06" x2="149.86" y2="99.06" width="0.1524" layer="91"/>
+<wire x1="149.86" y1="99.06" x2="149.86" y2="96.52" width="0.1524" layer="91"/>
+<label x="147.32" y="99.06" size="1.778" layer="95"/>
+</segment>
+</net>
+<net name="CTRL_OFF_1" class="0">
 <segment>
 <pinref part="CONTROLLER" gate="A" pin="O0"/>
@@
 <label x="-50.8" y="180.34" size="1.778" layer="95"/>
 </segment>
-</net>
-<net name="CTRL_ON_2" class="0">
+<segment>
+<pinref part="REGISTER_1_CLEAR_CX" gate="1" pin="1"/>
+<wire x1="114.3" y1="99.06" x2="101.6" y2="99.06" width="0.1524" layer="91"/>
+<label x="93.218" y="100.584" size="1.778" layer="95"/>
+</segment>
+</net>
+<net name="CTRL_OFF_2" class="0">
 <segment>
 <pinref part="CONTROLLER" gate="A" pin="O1"/>
@@
 </segment>
 </net>
-<net name="CTRL_ON_3" class="0">
+<net name="CTRL_OFF_3" class="0">
 <segment>
 <pinref part="CONTROLLER" gate="A" pin="O2"/>
@@
 </segment>
 </net>
-<net name="CTRL_ON_4" class="0">
+<net name="CTRL_OFF_4" class="0">
 <segment>
 <pinref part="CONTROLLER" gate="A" pin="O3"/>
@@
 <segment>
 <pinref part="CONTROLLER_INV_" gate="D" pin="I"/>
-<wire x1="25.4" y1="177.8" x2="10.16" y2="177.8" width="0.1524" layer="91"/>
+<wire x1="33.02" y1="177.8" x2="10.16" y2="177.8" width="0.1524" layer="91"/>
 <label x="17.78" y="177.8" size="1.778" layer="95"/>
 </segment>
 </net>
-<net name="CTRL_ON_5" class="0">
+<net name="CTRL_OFF_5" class="0">
 <segment>
 <pinref part="CONTROLLER" gate="A" pin="O4"/>
@@
 <segment>
 <pinref part="CONTROLLER_INV_" gate="E" pin="I"/>
-<wire x1="25.4" y1="190.5" x2="7.62" y2="190.5" width="0.1524" layer="91"/>
+<wire x1="33.02" y1="190.5" x2="7.62" y2="190.5" width="0.1524" layer="91"/>
 <wire x1="7.62" y1="190.5" x2="7.62" y2="187.96" width="0.1524" layer="91"/>
 <label x="17.78" y="187.96" size="1.778" layer="95"/>
 </segment>
 </net>
-<net name="CTRL_ON_6" class="0">
+<net name="CTRL_OFF_6" class="0">
 <segment>
 <pinref part="CONTROLLER" gate="A" pin="O5"/>
@@
 <segment>
 <pinref part="CONTROLLER_INV_" gate="F" pin="I"/>
-<wire x1="22.86" y1="205.74" x2="5.08" y2="205.74" width="0.1524" layer="91"/>
+<wire x1="30.48" y1="205.74" x2="5.08" y2="205.74" width="0.1524" layer="91"/>
 <label x="17.78" y="205.74" size="1.778" layer="95"/>
 </segment>
 </net>
-<net name="CTRL_ON_INV_3" class="0">
-<segment>
-<pinref part="CONTROLLER_INV_" gate="C" pin="O"/>
-<wire x1="-17.78" y1="208.28" x2="0" y2="208.28" width="0.1524" layer="91"/>
-<label x="-7.62" y="208.28" size="1.778" layer="95"/>
-</segment>
-</net>
-<net name="CTRL_ON_INV_2" class="0">
-<segment>
-<pinref part="CONTROLLER_INV_" gate="B" pin="O"/>
-<wire x1="-17.78" y1="193.04" x2="0" y2="193.04" width="0.1524" layer="91"/>
-<label x="-7.62" y="193.04" size="1.778" layer="95"/>
-</segment>
-</net>
-<net name="CTRL_ON_INV_1" class="0">
+<net name="CTRL_ON_1" class="0">
 <segment>
 <pinref part="CONTROLLER_INV_" gate="A" pin="O"/>
@@
 </segment>
 </net>
-<net name="CTRL_ON_INV_6" class="0">
-<segment>
-<pinref part="CONTROLLER_INV_" gate="F" pin="O"/>
-<wire x1="43.18" y1="205.74" x2="63.5" y2="205.74" width="0.1524" layer="91"/>
-<label x="58.42" y="205.74" size="1.778" layer="95"/>
-</segment>
-</net>
-<net name="CTRL_ON_INV_5" class="0">
-<segment>
-<pinref part="CONTROLLER_INV_" gate="E" pin="O"/>
-<wire x1="45.72" y1="190.5" x2="66.04" y2="190.5" width="0.1524" layer="91"/>
-<label x="66.04" y="190.5" size="1.778" layer="95"/>
-</segment>
-</net>
-<net name="CTRL_ON_INV_4" class="0">
-<segment>
-<pinref part="CONTROLLER_INV_" gate="D" pin="O"/>
-<wire x1="45.72" y1="177.8" x2="66.04" y2="177.8" width="0.1524" layer="91"/>
-<label x="66.04" y="180.34" size="1.778" layer="95"/>
-</segment>
-</net>
-<net name="N$2" class="0">
-<segment>
-<pinref part="REG_1_BIT_0_DIODE" gate="G$1" pin="A"/>
-<pinref part="REGISTER_1" gate="A" pin="Q1"/>
-<wire x1="137.16" y1="154.94" x2="124.46" y2="154.94" width="0.1524" layer="91"/>
-</segment>
-</net>
-<net name="N$3" class="0">
-<segment>
-<pinref part="REG_1_BIT_1_DIODE" gate="G$1" pin="A"/>
-<pinref part="REGISTER_1" gate="A" pin="Q2"/>
-<wire x1="129.54" y1="152.4" x2="124.46" y2="152.4" width="0.1524" layer="91"/>
-</segment>
-</net>
-<net name="N$4" class="0">
-<segment>
-<pinref part="REG_1_BIT_2_DIODE" gate="G$1" pin="A"/>
-<pinref part="REGISTER_1" gate="A" pin="Q3"/>
-<wire x1="139.7" y1="149.86" x2="124.46" y2="149.86" width="0.1524" layer="91"/>
-</segment>
-</net>
-<net name="N$5" class="0">
-<segment>
-<pinref part="REG_1_BIT_3_DIODE" gate="G$1" pin="A"/>
-<pinref part="REGISTER_1" gate="A" pin="Q4"/>
-<wire x1="129.54" y1="147.32" x2="124.46" y2="147.32" width="0.1524" layer="91"/>
-</segment>
-</net>
-<net name="REGISTER_1_CLK" class="0">
-<segment>
-<pinref part="REGISTER_1" gate="A" pin="CLK"/>
-<wire x1="99.06" y1="132.08" x2="83.82" y2="132.08" width="0.1524" layer="91"/>
-<label x="78.74" y="132.08" size="1.778" layer="95"/>
-</segment>
-</net>
-<net name="REGISTER_1_CLR" class="0">
-<segment>
-<pinref part="REGISTER_1" gate="A" pin="CLR"/>
-<wire x1="99.06" y1="129.54" x2="73.66" y2="129.54" width="0.1524" layer="91"/>
-<label x="76.2" y="127" size="1.778" layer="95"/>
-</segment>
-</net>

Commit message: Update fCPU
Parts:
- removed REG_1_BIT_0_DIODE, REG_1_BIT_1_DIODE, REG_1_BIT_2_DIODE, REG_1_BIT_3_DIODE: (no value), diode:DIODE-MELF-MLL41
- added INPUT_DEVICE_1, INPUT_DEVICE_2: (no value), special:SW_DIP-4
- added REGISTER_2: 74273N, 74xx-us:74273N
- added REGISTER_2_CLEAR_CX: (no value), microbuilder:SOLDERJUMPERREFLOW
- added RESISTOR_INPUT_DEVICES: (no value), resistor-sip:4610X
Connections:
- removed net N$2: REGISTER_1A.Q1, REG_1_BIT_0_DIODE.A
- removed net N$3: REGISTER_1A.Q2, REG_1_BIT_1_DIODE.A
- removed net N$4: REGISTER_1A.Q3, REG_1_BIT_2_DIODE.A
- removed net N$5: REGISTER_1A.Q4, REG_1_BIT_3_DIODE.A
- new net REGISTER_1_IN_BIT_0: INPUT_DEVICE_1.1, REGISTER_1A.D1, RESISTOR_INPUT_DEVICES.2
- new net REGISTER_1_IN_BIT_1: INPUT_DEVICE_1.2, REGISTER_1A.D2, RESISTOR_INPUT_DEVICES.3
- new net REGISTER_1_IN_BIT_2: INPUT_DEVICE_1.3, REGISTER_1A.D3, RESISTOR_INPUT_DEVICES.4
- new net REGISTER_1_IN_BIT_3: INPUT_DEVICE_1.4, REGISTER_1A.D4, RESISTOR_INPUT_DEVICES.5
- new net REGISTER_2_CLK: REGISTER_2A.CLK
- new net REGISTER_2_CLR: REGISTER_2A.CLR, REGISTER_2_CLEAR_CX.2
- new net REGISTER_2_IN_BIT_0: INPUT_DEVICE_2.1, REGISTER_2A.D1, RESISTOR_INPUT_DEVICES.6
- new net REGISTER_2_IN_BIT_1: INPUT_DEVICE_2.2, REGISTER_2A.D2, RESISTOR_INPUT_DEVICES.7
- new net REGISTER_2_IN_BIT_2: INPUT_DEVICE_2.3, REGISTER_2A.D3, RESISTOR_INPUT_DEVICES.8
- new net REGISTER_2_IN_BIT_3: INPUT_DEVICE_2.4, REGISTER_2A.D4, RESISTOR_INPUT_DEVICES.9
- net CTRL_OFF_2: now also REGISTER_2_CLEAR_CX.1
- net DTA_BUS_0: no longer REG_1_BIT_0_DIODE.C
- net DTA_BUS_1: no longer REG_1_BIT_1_DIODE.C
- net DTA_BUS_2: no longer REG_1_BIT_2_DIODE.C
- net DTA_BUS_3: no longer REG_1_BIT_3_DIODE.C
- net GND: now also REGISTER_1A.D5, REGISTER_1A.D6, REGISTER_1A.D7, REGISTER_1A.D8, REGISTER_2A.D5, REGISTER_2A.D6, REGISTER_2A.D7, REGISTER_2A.D8, RESISTOR_INPUT_DEVICES.1
- net VCC: now also INPUT_DEVICE_1.5, INPUT_DEVICE_1.6, INPUT_DEVICE_1.7, INPUT_DEVICE_1.8, INPUT_DEVICE_2.5, INPUT_DEVICE_2.6, INPUT_DEVICE_2.7, INPUT_DEVICE_2.8
Other:
- moved on the sheet: REGISTER_1_CLEAR_CX

Commit message: Update fCPU
Parts:
- removed CONTROLLER: 74LS42N, 74xx-us:74LS42N
- removed PRG_COUNTER: 74LS90N, 74xx-us:74LS90N
- added ADDER_74LS283N: 74LS283N, 74xx-us:74LS283N
- added CONTROLLER_CD4017BE: CD4017, SparkFun-DigitalIC:CD4017
- renumbered CONTROLLER_INV_ to CONTROLLER_INV_SN74LS14, DISPLAY_DRIVER to DISPLAY_DRIVER_74LS47, REGISTER_1 to REGISTER_1_SN74LS273, REGISTER_2 to REGISTER_2_SN74LS273
Connections:
- net CTRL_ON_3 renamed CTRL_LOW_3
- net CTRL_ON_4 renamed CTRL_LOW_4
- net CTRL_ON_5 renamed CTRL_LOW_5
- net CTRL_ON_6 renamed CTRL_LOW_6
- removed net CTRL_OFF_1: CONTROLLERA.O0, CONTROLLER_INV_SN74LS14A.I, REGISTER_1_CLEAR_CX.1
- removed net CTRL_OFF_2: CONTROLLERA.O1, CONTROLLER_INV_SN74LS14B.I, REGISTER_2_CLEAR_CX.1
- removed net CTRL_OFF_3: CONTROLLERA.O2, CONTROLLER_INV_SN74LS14C.I
- removed net CTRL_OFF_4: CONTROLLERA.O3, CONTROLLER_INV_SN74LS14D.I
- removed net CTRL_OFF_5: CONTROLLERA.O4, CONTROLLER_INV_SN74LS14E.I
- removed net CTRL_OFF_6: CONTROLLERA.O5, CONTROLLER_INV_SN74LS14F.I
- removed net CTRL_ON_1: CONTROLLER_INV_SN74LS14A.O
- removed net CTRL_ON_2: CONTROLLER_INV_SN74LS14B.O
- removed net PC_0: CONTROLLERA.A, PRG_COUNTERA.CKB, PRG_COUNTERA.QA
- removed net PC_1: CONTROLLERA.B, PRG_COUNTERA.QB
- removed net PC_2: CONTROLLERA.C, PRG_COUNTERA.QC
- removed net PC_3: CONTROLLERA.D, PRG_COUNTERA.QD
- new net CTRL_HIGH_1: CONTROLLER_CD4017BEA.Q0, CONTROLLER_INV_SN74LS14A.I
- new net CTRL_HIGH_2: CONTROLLER_CD4017BEA.Q1, CONTROLLER_INV_SN74LS14B.I
- new net CTRL_HIGH_3: CONTROLLER_CD4017BEA.Q2, CONTROLLER_INV_SN74LS14C.I
- new net CTRL_HIGH_4: CONTROLLER_CD4017BEA.Q3, CONTROLLER_INV_SN74LS14D.I
- new net CTRL_HIGH_5: CONTROLLER_CD4017BEA.Q4, CONTROLLER_INV_SN74LS14E.I
- new net CTRL_HIGH_6: CONTROLLER_CD4017BEA.Q5, CONTROLLER_INV_SN74LS14F.I
- new net CTRL_LOW_1: CONTROLLER_INV_SN74LS14A.O, REGISTER_1_CLEAR_CX.1
- new net CTRL_LOW_2: CONTROLLER_INV_SN74LS14B.O, REGISTER_2_CLEAR_CX.1
- new net N$10: ADDER_74LS283NA.S1
- new net N$11: ADDER_74LS283NA.S2
- new net N$12: ADDER_74LS283NA.S3
- new net N$13: ADDER_74LS283NA.S4
- new net REGISTER_1_OUT_BIT_0: ADDER_74LS283NA.A1, REGISTER_1_SN74LS273A.Q1
- new net REGISTER_1_OUT_BIT_1: ADDER_74LS283NA.A2, REGISTER_1_SN74LS273A.Q2
- new net REGISTER_1_OUT_BIT_2: ADDER_74LS283NA.A3, REGISTER_1_SN74LS273A.Q3
- new net REGISTER_1_OUT_BIT_3: ADDER_74LS283NA.A4, REGISTER_1_SN74LS273A.Q4
- new net REGISTER_2_OUT_BIT_0: ADDER_74LS283NA.B1, REGISTER_2_SN74LS273A.Q1
- new net REGISTER_2_OUT_BIT_1: ADDER_74LS283NA.B2, REGISTER_2_SN74LS273A.Q2
- new net REGISTER_2_OUT_BIT_2: ADDER_74LS283NA.B3, REGISTER_2_SN74LS273A.Q3
- new net REGISTER_2_OUT_BIT_3: ADDER_74LS283NA.B4, REGISTER_2_SN74LS273A.Q4
- net GND: now also ADDER_74LS283NA.C0, CONTROLLER_CD4017BEA.ENA, CONTROLLER_CD4017BEA.RES; no longer PRG_COUNTERA.R0(1), PRG_COUNTERA.R0(2), PRG_COUNTERA.R9(1), PRG_COUNTERA.R9(2)
- net TMR555_OUTPUT: now also CONTROLLER_CD4017BEA.CLK; no longer PRG_COUNTERA.CKA

Commit message: Update fCPU
Parts:
- removed CONTROLLER_CD4017BE: CD4017, SparkFun-DigitalIC:CD4017
- removed CONTROLLER_INV_SN74LS14: 74LS14N, 74xx-us:74LS14N
- removed REGISTER_1_CLEAR_CX, REGISTER_2_CLEAR_CX: (no value), microbuilder:SOLDERJUMPERREFLOW
- added CLEAR_REGISTER_1, CLEAR_REGISTER_2, CLOCK_REGISTER_1, CLOCK_REGISTER_2: (no value), switch-omron:10-XX
- added INPUT_DEVICE_1_EX, INPUT_DEVICE_2_EX: (no value), pinhead:PINHD-1X4
- added LED_POWER: (no value), adafruit:LEDSMT1206
- added RESISTOR_SWITCHES: (no value), resistor-sip:4610X
Connections:
- removed net CTRL_HIGH_1: CONTROLLER_CD4017BEA.Q0, CONTROLLER_INV_SN74LS14A.I
- removed net CTRL_HIGH_2: CONTROLLER_CD4017BEA.Q1, CONTROLLER_INV_SN74LS14B.I
- removed net CTRL_HIGH_3: CONTROLLER_CD4017BEA.Q2, CONTROLLER_INV_SN74LS14C.I
- removed net CTRL_HIGH_4: CONTROLLER_CD4017BEA.Q3, CONTROLLER_INV_SN74LS14D.I
- removed net CTRL_HIGH_5: CONTROLLER_CD4017BEA.Q4, CONTROLLER_INV_SN74LS14E.I
- removed net CTRL_HIGH_6: CONTROLLER_CD4017BEA.Q5, CONTROLLER_INV_SN74LS14F.I
- removed net CTRL_LOW_1: CONTROLLER_INV_SN74LS14A.O, REGISTER_1_CLEAR_CX.1
- removed net CTRL_LOW_2: CONTROLLER_INV_SN74LS14B.O, REGISTER_2_CLEAR_CX.1
- removed net CTRL_LOW_3: CONTROLLER_INV_SN74LS14C.O
- removed net CTRL_LOW_4: CONTROLLER_INV_SN74LS14D.O
- removed net CTRL_LOW_5: CONTROLLER_INV_SN74LS14E.O
- removed net CTRL_LOW_6: CONTROLLER_INV_SN74LS14F.O
- removed net N$10: ADDER_74LS283NA.S1
- removed net N$11: ADDER_74LS283NA.S2
- removed net N$12: ADDER_74LS283NA.S3
- removed net N$13: ADDER_74LS283NA.S4
- new net CLEAR_REGISTER_1_TO_GND: CLEAR_REGISTER_1.S, RESISTOR_SWITCHES.4
- new net CLEAR_REGISTER_2_TO_GND: CLEAR_REGISTER_2.S, RESISTOR_SWITCHES.5
- new net LED_POWER_TO_GND: LED_POWER.C, RESISTOR_SWITCHES.9
- net DTA_BUS_0: now also ADDER_74LS283NA.S1
- net DTA_BUS_1: now also ADDER_74LS283NA.S2
- net DTA_BUS_2: now also ADDER_74LS283NA.S3
- net DTA_BUS_3: now also ADDER_74LS283NA.S4
- net GND: now also RESISTOR_SWITCHES.1; no longer CONTROLLER_CD4017BEA.ENA, CONTROLLER_CD4017BEA.RES
- net REGISTER_1_CLK: now also CLOCK_REGISTER_1.P1, RESISTOR_SWITCHES.2
- net REGISTER_1_CLR: now also CLEAR_REGISTER_1.P1; no longer REGISTER_1_CLEAR_CX.2
- net REGISTER_1_IN_BIT_0: now also INPUT_DEVICE_1_EX.1
- net REGISTER_1_IN_BIT_1: now also INPUT_DEVICE_1_EX.2
- net REGISTER_1_IN_BIT_2: now also INPUT_DEVICE_1_EX.3
- net REGISTER_1_IN_BIT_3: now also INPUT_DEVICE_1_EX.4
- net REGISTER_2_CLK: now also CLOCK_REGISTER_2.P1, RESISTOR_SWITCHES.3
- net REGISTER_2_CLR: now also CLEAR_REGISTER_2.P1; no longer REGISTER_2_CLEAR_CX.2
- net REGISTER_2_IN_BIT_0: now also INPUT_DEVICE_2_EX.1
- net REGISTER_2_IN_BIT_1: now also INPUT_DEVICE_2_EX.2
- net REGISTER_2_IN_BIT_2: now also INPUT_DEVICE_2_EX.3
- net REGISTER_2_IN_BIT_3: now also INPUT_DEVICE_2_EX.4
- net TMR555_OUTPUT: now also LED_POWER.A; no longer CONTROLLER_CD4017BEA.CLK
- net VCC: now also CLOCK_REGISTER_1.S, CLOCK_REGISTER_2.S
