File: EXTENSIONS/Analog/fCPU/bu/fCPU.sch (EAGLE design)
At the start: 19 parts

Commit message: Update fCPU
Parts:
- removed INPUT_DEVICE_1_EX, INPUT_DEVICE_2_EX: (no value), pinhead:PINHD-1X4
- added EXTERNAL_CONTROL: (no value), adafruit:PINHD-1X12
Connections:
- net REGISTER_1_CLK: now also EXTERNAL_CONTROL.9
- net REGISTER_1_CLR: now also EXTERNAL_CONTROL.10
- net REGISTER_1_IN_BIT_0: now also EXTERNAL_CONTROL.1; no longer INPUT_DEVICE_1_EX.1
- net REGISTER_1_IN_BIT_1: now also EXTERNAL_CONTROL.2; no longer INPUT_DEVICE_1_EX.2
- net REGISTER_1_IN_BIT_2: now also EXTERNAL_CONTROL.3; no longer INPUT_DEVICE_1_EX.3
- net REGISTER_1_IN_BIT_3: now also EXTERNAL_CONTROL.4; no longer INPUT_DEVICE_1_EX.4
- net REGISTER_2_CLK: now also EXTERNAL_CONTROL.11
- net REGISTER_2_CLR: now also EXTERNAL_CONTROL.12
- net REGISTER_2_IN_BIT_0: now also EXTERNAL_CONTROL.5; no longer INPUT_DEVICE_2_EX.1
- net REGISTER_2_IN_BIT_1: now also EXTERNAL_CONTROL.6; no longer INPUT_DEVICE_2_EX.2
- net REGISTER_2_IN_BIT_2: now also EXTERNAL_CONTROL.7; no longer INPUT_DEVICE_2_EX.3
- net REGISTER_2_IN_BIT_3: now also EXTERNAL_CONTROL.8; no longer INPUT_DEVICE_2_EX.4
Changed lines of the file:
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@@
 <part name="CLEAR_REGISTER_2" library="switch-omron" deviceset="10-XX" device=""/>
 <part name="LED_POWER" library="adafruit" deviceset="LED" device="SMT1206"/>
-<part name="INPUT_DEVICE_1_EX" library="pinhead" deviceset="PINHD-1X4" device=""/>
-<part name="INPUT_DEVICE_2_EX" library="pinhead" deviceset="PINHD-1X4" device=""/>
+<part name="EXTERNAL_CONTROL" library="adafruit" deviceset="PINHD-1X12" device=""/>
 </parts>
 <sheets>
@@
 <instance part="CLEAR_REGISTER_2" gate="1" x="-45.72" y="132.08"/>
 <instance part="LED_POWER" gate="G$1" x="78.74" y="193.04"/>
-<instance part="INPUT_DEVICE_1_EX" gate="A" x="289.56" y="152.4" smashed="yes" rot="R180">
-<attribute name="NAME" x="306.07" y="144.145" size="1.778" layer="95" rot="R180"/>
-<attribute name="VALUE" x="295.91" y="160.02" size="1.778" layer="96" rot="R180"/>
-</instance>
-<instance part="INPUT_DEVICE_2_EX" gate="A" x="289.56" y="132.08" smashed="yes" rot="R180">
-<attribute name="NAME" x="306.07" y="123.825" size="1.778" layer="95" rot="R180"/>
-<attribute name="VALUE" x="295.91" y="139.7" size="1.778" layer="96" rot="R180"/>
-</instance>
+<instance part="EXTERNAL_CONTROL" gate="G$1" x="284.48" y="96.52" rot="R180"/>
 </instances>
 <busses>
@@
 <label x="40.64" y="175.26" size="1.778" layer="95" rot="R270"/>
 </segment>
+<segment>
+<pinref part="EXTERNAL_CONTROL" gate="G$1" pin="9"/>
+<wire x1="287.02" y1="104.14" x2="320.04" y2="104.14" width="0.1524" layer="91"/>
+<label x="320.04" y="104.14" size="1.778" layer="95"/>
+</segment>
 </net>
 <net name="REGISTER_1_CLR" class="0">
@@
 <wire x1="-17.78" y1="132.08" x2="-17.78" y2="127" width="0.1524" layer="91"/>
 </segment>
+<segment>
+<pinref part="EXTERNAL_CONTROL" gate="G$1" pin="10"/>
+<wire x1="287.02" y1="106.68" x2="322.58" y2="106.68" width="0.1524" layer="91"/>
+<label x="320.04" y="106.68" size="1.778" layer="95"/>
+</segment>
 </net>
 <net name="REGISTER_2_CLK" class="0">
@@
 <label x="43.18" y="177.8" size="1.778" layer="95" rot="R270"/>
 </segment>
+<segment>
+<pinref part="EXTERNAL_CONTROL" gate="G$1" pin="11"/>
+<wire x1="287.02" y1="109.22" x2="320.04" y2="109.22" width="0.1524" layer="91"/>
+<label x="320.04" y="109.22" size="1.778" layer="95"/>
+</segment>
 </net>
 <net name="REGISTER_2_CLR" class="0">
@@
 <label x="-39.878" y="100.33" size="1.778" layer="95" rot="R90"/>
 </segment>
+<segment>
+<pinref part="EXTERNAL_CONTROL" gate="G$1" pin="12"/>
+<wire x1="287.02" y1="111.76" x2="317.5" y2="111.76" width="0.1524" layer="91"/>
+<label x="317.5" y="111.76" size="1.778" layer="95"/>
+</segment>
 </net>
 <net name="REGISTER_1_IN_BIT_0" class="0">
@@
 </segment>
 <segment>
-<pinref part="INPUT_DEVICE_1_EX" gate="A" pin="1"/>
-<wire x1="292.1" y1="147.32" x2="309.88" y2="147.32" width="0.1524" layer="91"/>
-<label x="321.564" y="148.844" size="1.778" layer="95" rot="R180"/>
+<pinref part="EXTERNAL_CONTROL" gate="G$1" pin="1"/>
+<wire x1="287.02" y1="83.82" x2="322.58" y2="83.82" width="0.1524" layer="91"/>
+<label x="320.04" y="83.82" size="1.778" layer="95"/>
 </segment>
 </net>
@@
 </segment>
 <segment>
-<pinref part="INPUT_DEVICE_1_EX" gate="A" pin="2"/>
-<wire x1="292.1" y1="149.86" x2="309.88" y2="149.86" width="0.1524" layer="91"/>
-<label x="322.326" y="151.638" size="1.778" layer="95" rot="R180"/>
+<pinref part="EXTERNAL_CONTROL" gate="G$1" pin="2"/>
+<wire x1="287.02" y1="86.36" x2="322.58" y2="86.36" width="0.1524" layer="91"/>
+<label x="320.04" y="86.36" size="1.778" layer="95"/>
 </segment>
 </net>
@@
 </segment>
 <segment>
-<pinref part="INPUT_DEVICE_1_EX" gate="A" pin="3"/>
-<wire x1="292.1" y1="152.4" x2="307.34" y2="152.4" width="0.1524" layer="91"/>
-<label x="321.564" y="154.178" size="1.778" layer="95" rot="R180"/>
+<pinref part="EXTERNAL_CONTROL" gate="G$1" pin="3"/>
+<wire x1="287.02" y1="88.9" x2="320.04" y2="88.9" width="0.1524" layer="91"/>
+<label x="320.04" y="88.9" size="1.778" layer="95"/>
 </segment>
 </net>
@@
 </segment>
 <segment>
-<pinref part="INPUT_DEVICE_1_EX" gate="A" pin="4"/>
-<wire x1="292.1" y1="154.94" x2="317.5" y2="154.94" width="0.1524" layer="91"/>
-<label x="321.818" y="157.988" size="1.778" layer="95" rot="R180"/>
+<pinref part="EXTERNAL_CONTROL" gate="G$1" pin="4"/>
+<wire x1="287.02" y1="91.44" x2="322.58" y2="91.44" width="0.1524" layer="91"/>
+<label x="320.04" y="91.44" size="1.778" layer="95"/>
 </segment>
 </net>
@@
 </segment>
 <segment>
-<pinref part="INPUT_DEVICE_2_EX" gate="A" pin="1"/>
-<wire x1="292.1" y1="127" x2="314.96" y2="127" width="0.1524" layer="91"/>
-<label x="312.42" y="127" size="1.778" layer="95"/>
+<pinref part="EXTERNAL_CONTROL" gate="G$1" pin="5"/>
+<wire x1="287.02" y1="93.98" x2="322.58" y2="93.98" width="0.1524" layer="91"/>
+<label x="320.04" y="93.98" size="1.778" layer="95"/>
 </segment>
 </net>
@@
 </segment>
 <segment>
-<pinref part="INPUT_DEVICE_2_EX" gate="A" pin="2"/>
-<wire x1="292.1" y1="129.54" x2="314.96" y2="129.54" width="0.1524" layer="91"/>
-<label x="312.42" y="129.54" size="1.778" layer="95"/>
+<pinref part="EXTERNAL_CONTROL" gate="G$1" pin="6"/>
+<wire x1="287.02" y1="96.52" x2="322.58" y2="96.52" width="0.1524" layer="91"/>
+<label x="320.04" y="96.52" size="1.778" layer="95"/>
 </segment>
 </net>
@@
 </segment>
 <segment>
-<pinref part="INPUT_DEVICE_2_EX" gate="A" pin="3"/>
-<wire x1="292.1" y1="132.08" x2="314.96" y2="132.08" width="0.1524" layer="91"/>
-<label x="312.42" y="132.08" size="1.778" layer="95"/>
+<pinref part="EXTERNAL_CONTROL" gate="G$1" pin="7"/>
+<wire x1="287.02" y1="99.06" x2="320.04" y2="99.06" width="0.1524" layer="91"/>
+<label x="320.04" y="99.06" size="1.778" layer="95"/>
 </segment>
 </net>
@@
 </segment>
 <segment>
-<pinref part="INPUT_DEVICE_2_EX" gate="A" pin="4"/>
-<wire x1="292.1" y1="134.62" x2="314.96" y2="134.62" width="0.1524" layer="91"/>
-<label x="312.42" y="134.62" size="1.778" layer="95"/>
-</segment>
-</net>
+<pinref part="EXTERNAL_CONTROL" gate="G$1" pin="8"/>
+<wire x1="287.02" y1="101.6" x2="322.58" y2="101.6" width="0.1524" layer="91"/>
+<label x="320.04" y="101.6" size="1.778" layer="95"/>
+</segment>
+</net>

Commit message: Update fCPU
Connections:
- net TMR555_OUTPUT: no longer LED_POWER.A
- net VCC: now also LED_POWER.A
Changed lines of the file:
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@@
 <label x="-27.94" y="213.36" size="1.778" layer="95"/>
+</segment>
+<segment>
+<pinref part="LED_POWER" gate="G$1" pin="A"/>
+<wire x1="78.74" y1="195.58" x2="78.74" y2="205.74" width="0.1524" layer="91"/>
+<label x="78.74" y="203.2" size="1.778" layer="95"/>
 </segment>
 </net>
@@
 <label x="33.02" y="104.14" size="1.778" layer="95"/>
 </segment>
-<segment>
-<pinref part="LED_POWER" gate="G$1" pin="A"/>
-<wire x1="78.74" y1="195.58" x2="78.74" y2="205.74" width="0.1524" layer="91"/>
-<label x="78.74" y="203.2" size="1.778" layer="95"/>
-</segment>
 </net>

Commit message: Update fCPU
Parts:
- renumbered EXTERNAL_CONTROL to EXTERNAL_CONTROL_INPUT, R_100O_0 to R_100_O
Changed lines of the file:
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@@
 <part name="OUTPUTS" library="pinhead" deviceset="PINHD-1X4" device=""/>
 <part name="GND2" library="supply1" deviceset="GND" device=""/>
-<part name="R_100O_0" library="adafruit" deviceset="R-US_" device="R1206"/>
+<part name="R_100_O" library="adafruit" deviceset="R-US_" device="R1206"/>
 <part name="DISPLAY_DRIVER_74LS47" library="74xx-us" deviceset="74*47" device="N" technology="LS"/>
 <part name="DIGIT_0_ANODE" library="special" deviceset="7SEG-CA" device=""/>
@@
 <part name="CLEAR_REGISTER_2" library="switch-omron" deviceset="10-XX" device=""/>
 <part name="LED_POWER" library="adafruit" deviceset="LED" device="SMT1206"/>
-<part name="EXTERNAL_CONTROL" library="adafruit" deviceset="PINHD-1X12" device=""/>
+<part name="EXTERNAL_CONTROL_INPUT" library="adafruit" deviceset="PINHD-1X12" device=""/>
 </parts>
 <sheets>
@@
 <instance part="OUTPUTS" gate="A" x="17.78" y="104.14" rot="R180"/>
 <instance part="GND2" gate="1" x="43.18" y="99.06" rot="R90"/>
-<instance part="R_100O_0" gate="G$1" x="50.8" y="71.12"/>
+<instance part="R_100_O" gate="G$1" x="50.8" y="71.12"/>
 <instance part="DISPLAY_DRIVER_74LS47" gate="G$1" x="-50.8" y="50.8"/>
 <instance part="DIGIT_0_ANODE" gate="G$1" x="25.4" y="76.2"/>
@@
 <instance part="CLEAR_REGISTER_2" gate="1" x="-45.72" y="132.08"/>
 <instance part="LED_POWER" gate="G$1" x="78.74" y="193.04"/>
-<instance part="EXTERNAL_CONTROL" gate="G$1" x="284.48" y="96.52" rot="R180"/>
+<instance part="EXTERNAL_CONTROL_INPUT" gate="G$1" x="284.48" y="96.52" rot="R180"/>
 </instances>
 <busses>
@@
 </segment>
 <segment>
-<pinref part="R_100O_0" gate="G$1" pin="2"/>
+<pinref part="R_100_O" gate="G$1" pin="2"/>
 <wire x1="55.88" y1="71.12" x2="71.12" y2="71.12" width="0.1524" layer="91"/>
 <label x="60.96" y="71.12" size="1.778" layer="95"/>
@@
 <segment>
 <pinref part="DIGIT_0_ANODE" gate="G$1" pin="CA2"/>
-<pinref part="R_100O_0" gate="G$1" pin="1"/>
+<pinref part="R_100_O" gate="G$1" pin="1"/>
 <wire x1="33.02" y1="71.12" x2="45.72" y2="71.12" width="0.1524" layer="91"/>
 </segment>
@@
 </segment>
 <segment>
-<pinref part="EXTERNAL_CONTROL" gate="G$1" pin="9"/>
+<pinref part="EXTERNAL_CONTROL_INPUT" gate="G$1" pin="9"/>
 <wire x1="287.02" y1="104.14" x2="320.04" y2="104.14" width="0.1524" layer="91"/>
 <label x="320.04" y="104.14" size="1.778" layer="95"/>
@@
 </segment>
 <segment>
-<pinref part="EXTERNAL_CONTROL" gate="G$1" pin="10"/>
+<pinref part="EXTERNAL_CONTROL_INPUT" gate="G$1" pin="10"/>
 <wire x1="287.02" y1="106.68" x2="322.58" y2="106.68" width="0.1524" layer="91"/>
 <label x="320.04" y="106.68" size="1.778" layer="95"/>
@@
 </segment>
 <segment>
-<pinref part="EXTERNAL_CONTROL" gate="G$1" pin="11"/>
+<pinref part="EXTERNAL_CONTROL_INPUT" gate="G$1" pin="11"/>
 <wire x1="287.02" y1="109.22" x2="320.04" y2="109.22" width="0.1524" layer="91"/>
 <label x="320.04" y="109.22" size="1.778" layer="95"/>
@@
 </segment>
 <segment>
-<pinref part="EXTERNAL_CONTROL" gate="G$1" pin="12"/>
+<pinref part="EXTERNAL_CONTROL_INPUT" gate="G$1" pin="12"/>
 <wire x1="287.02" y1="111.76" x2="317.5" y2="111.76" width="0.1524" layer="91"/>
 <label x="317.5" y="111.76" size="1.778" layer="95"/>
@@
 </segment>
 <segment>
-<pinref part="EXTERNAL_CONTROL" gate="G$1" pin="1"/>
+<pinref part="EXTERNAL_CONTROL_INPUT" gate="G$1" pin="1"/>
 <wire x1="287.02" y1="83.82" x2="322.58" y2="83.82" width="0.1524" layer="91"/>
 <label x="320.04" y="83.82" size="1.778" layer="95"/>
@@
 </segment>
 <segment>
-<pinref part="EXTERNAL_CONTROL" gate="G$1" pin="2"/>
+<pinref part="EXTERNAL_CONTROL_INPUT" gate="G$1" pin="2"/>
 <wire x1="287.02" y1="86.36" x2="322.58" y2="86.36" width="0.1524" layer="91"/>
 <label x="320.04" y="86.36" size="1.778" layer="95"/>
@@
 </segment>
 <segment>
-<pinref part="EXTERNAL_CONTROL" gate="G$1" pin="3"/>
+<pinref part="EXTERNAL_CONTROL_INPUT" gate="G$1" pin="3"/>
 <wire x1="287.02" y1="88.9" x2="320.04" y2="88.9" width="0.1524" layer="91"/>
 <label x="320.04" y="88.9" size="1.778" layer="95"/>
@@
 </segment>
 <segment>
-<pinref part="EXTERNAL_CONTROL" gate="G$1" pin="4"/>
+<pinref part="EXTERNAL_CONTROL_INPUT" gate="G$1" pin="4"/>
 <wire x1="287.02" y1="91.44" x2="322.58" y2="91.44" width="0.1524" layer="91"/>
 <label x="320.04" y="91.44" size="1.778" layer="95"/>
@@
 </segment>
 <segment>
-<pinref part="EXTERNAL_CONTROL" gate="G$1" pin="5"/>
+<pinref part="EXTERNAL_CONTROL_INPUT" gate="G$1" pin="5"/>
 <wire x1="287.02" y1="93.98" x2="322.58" y2="93.98" width="0.1524" layer="91"/>
 <label x="320.04" y="93.98" size="1.778" layer="95"/>
@@
 </segment>
 <segment>
-<pinref part="EXTERNAL_CONTROL" gate="G$1" pin="6"/>
+<pinref part="EXTERNAL_CONTROL_INPUT" gate="G$1" pin="6"/>
 <wire x1="287.02" y1="96.52" x2="322.58" y2="96.52" width="0.1524" layer="91"/>
 <label x="320.04" y="96.52" size="1.778" layer="95"/>
@@
 </segment>
 <segment>
-<pinref part="EXTERNAL_CONTROL" gate="G$1" pin="7"/>
+<pinref part="EXTERNAL_CONTROL_INPUT" gate="G$1" pin="7"/>
 <wire x1="287.02" y1="99.06" x2="320.04" y2="99.06" width="0.1524" layer="91"/>
 <label x="320.04" y="99.06" size="1.778" layer="95"/>
@@
 </segment>
 <segment>
-<pinref part="EXTERNAL_CONTROL" gate="G$1" pin="8"/>
+<pinref part="EXTERNAL_CONTROL_INPUT" gate="G$1" pin="8"/>
 <wire x1="287.02" y1="101.6" x2="322.58" y2="101.6" width="0.1524" layer="91"/>
 <label x="320.04" y="101.6" size="1.778" layer="95"/>
