File: USB.BusinessCard/bu/USB.BusinessCard.sch (EAGLE design)
At the start: 5 parts

Commit message: Write firmware for Usb Business Card
Parts:
- removed JP2: (no value), adafruit:PINHD-1X1
- added JP_I2C_OLED_SSD1306: (no value), pinhead:PINHD-1X4
- renumbered JP_LEFT to ARDUINO_PRO_MINI_LEFT, JP_RIGHT to ARDUINO_PRO_MINI_RIGHT
Connections:
- net A4_I2C_SDA: now also JP_I2C_OLED_SSD1306.4; no longer JP2.1
- net A5_I2C_SCL: now also JP_I2C_OLED_SSD1306.3
- net GND: now also JP_I2C_OLED_SSD1306.1
- net VCC: now also JP_I2C_OLED_SSD1306.2
Changed lines of the file:
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@@
 <part name="GND2" library="supply1" deviceset="GND" device=""/>
 <part name="JP1" library="SparkFun-Connectors" deviceset="USB" device="PCB"/>
-<part name="JP_LEFT" library="adafruit" deviceset="PINHD-1X12" device=""/>
+<part name="ARDUINO_PRO_MINI_LEFT" library="adafruit" deviceset="PINHD-1X12" device=""/>
 <part name="GND3" library="supply1" deviceset="GND" device=""/>
-<part name="JP_RIGHT" library="adafruit" deviceset="PINHD-1X12" device=""/>
+<part name="ARDUINO_PRO_MINI_RIGHT" library="adafruit" deviceset="PINHD-1X12" device=""/>
 <part name="GND4" library="supply1" deviceset="GND" device=""/>
 <part name="JP_TOP" library="pinhead" deviceset="PINHD-1X4" device=""/>
-<part name="JP2" library="adafruit" deviceset="PINHD-1X1" device=""/>
+<part name="JP_I2C_OLED_SSD1306" library="pinhead" deviceset="PINHD-1X4" device=""/>
+<part name="GND5" library="supply1" deviceset="GND" device=""/>
 </parts>
 <sheets>
@@
 <instance part="GND2" gate="1" x="119.38" y="45.72"/>
 <instance part="JP1" gate="G$1" x="-5.08" y="86.36" rot="R180"/>
-<instance part="JP_LEFT" gate="G$1" x="63.5" y="83.82"/>
+<instance part="ARDUINO_PRO_MINI_LEFT" gate="G$1" x="63.5" y="83.82"/>
 <instance part="GND3" gate="1" x="33.02" y="71.12" rot="R270"/>
-<instance part="JP_RIGHT" gate="G$1" x="114.3" y="83.82"/>
+<instance part="ARDUINO_PRO_MINI_RIGHT" gate="G$1" x="114.3" y="83.82"/>
 <instance part="GND4" gate="1" x="83.82" y="76.2" rot="R270"/>
 <instance part="JP_TOP" gate="A" x="81.28" y="43.18" rot="R270"/>
-<instance part="JP2" gate="G$1" x="5.08" y="60.96" rot="R180"/>
+<instance part="JP_I2C_OLED_SSD1306" gate="A" x="40.64" y="43.18"/>
+<instance part="GND5" gate="1" x="12.7" y="48.26" rot="R270"/>
 </instances>
 <busses>
@@
 </segment>
 <segment>
-<pinref part="JP_LEFT" gate="G$1" pin="11"/>
+<pinref part="ARDUINO_PRO_MINI_LEFT" gate="G$1" pin="11"/>
 <pinref part="GND3" gate="1" pin="GND"/>
 <wire x1="60.96" y1="71.12" x2="35.56" y2="71.12" width="0.1524" layer="91"/>
 </segment>
 <segment>
-<pinref part="JP_RIGHT" gate="G$1" pin="9"/>
+<pinref part="ARDUINO_PRO_MINI_RIGHT" gate="G$1" pin="9"/>
 <pinref part="GND4" gate="1" pin="GND"/>
 <wire x1="111.76" y1="76.2" x2="86.36" y2="76.2" width="0.1524" layer="91"/>
+</segment>
+<segment>
+<pinref part="JP_I2C_OLED_SSD1306" gate="A" pin="1"/>
+<pinref part="GND5" gate="1" pin="GND"/>
+<wire x1="38.1" y1="48.26" x2="15.24" y2="48.26" width="0.1524" layer="91"/>
 </segment>
 </net>
@@
 </segment>
 <segment>
-<pinref part="JP_LEFT" gate="G$1" pin="9"/>
+<pinref part="ARDUINO_PRO_MINI_LEFT" gate="G$1" pin="9"/>
 <wire x1="60.96" y1="76.2" x2="48.26" y2="76.2" width="0.1524" layer="91"/>
 <label x="48.26" y="76.2" size="1.778" layer="95"/>
 </segment>
+<segment>
+<pinref part="JP_I2C_OLED_SSD1306" gate="A" pin="2"/>
+<wire x1="38.1" y1="45.72" x2="17.78" y2="45.72" width="0.1524" layer="91"/>
+<label x="17.78" y="45.72" size="1.778" layer="95"/>
+</segment>
 </net>
 <net name="RAW" class="0">
 <segment>
-<pinref part="JP_LEFT" gate="G$1" pin="12"/>
+<pinref part="ARDUINO_PRO_MINI_LEFT" gate="G$1" pin="12"/>
 <wire x1="60.96" y1="68.58" x2="43.18" y2="68.58" width="0.1524" layer="91"/>
 <label x="43.18" y="68.58" size="1.778" layer="95"/>
@@
 <net name="RST" class="0">
 <segment>
-<pinref part="JP_LEFT" gate="G$1" pin="10"/>
+<pinref part="ARDUINO_PRO_MINI_LEFT" gate="G$1" pin="10"/>
 <wire x1="60.96" y1="73.66" x2="35.56" y2="73.66" width="0.1524" layer="91"/>
 <label x="35.56" y="73.66" size="1.778" layer="95"/>
 </segment>
 <segment>
-<pinref part="JP_RIGHT" gate="G$1" pin="10"/>
+<pinref part="ARDUINO_PRO_MINI_RIGHT" gate="G$1" pin="10"/>
 <wire x1="111.76" y1="73.66" x2="91.44" y2="73.66" width="0.1524" layer="91"/>
 <label x="93.98" y="73.66" size="1.778" layer="95"/>
@@
 <net name="A3" class="0">
 <segment>
-<pinref part="JP_LEFT" gate="G$1" pin="8"/>
+<pinref part="ARDUINO_PRO_MINI_LEFT" gate="G$1" pin="8"/>
 <wire x1="60.96" y1="78.74" x2="35.56" y2="78.74" width="0.1524" layer="91"/>
 <label x="35.56" y="78.74" size="1.778" layer="95"/>
@@
 <net name="A2" class="0">
 <segment>
-<pinref part="JP_LEFT" gate="G$1" pin="7"/>
+<pinref part="ARDUINO_PRO_MINI_LEFT" gate="G$1" pin="7"/>
 <wire x1="60.96" y1="81.28" x2="48.26" y2="81.28" width="0.1524" layer="91"/>
 <label x="48.26" y="81.28" size="1.778" layer="95"/>
@@
 <net name="A1" class="0">
 <segment>
-<pinref part="JP_LEFT" gate="G$1" pin="6"/>
+<pinref part="ARDUINO_PRO_MINI_LEFT" gate="G$1" pin="6"/>
 <wire x1="60.96" y1="83.82" x2="35.56" y2="83.82" width="0.1524" layer="91"/>
 <label x="35.56" y="83.82" size="1.778" layer="95"/>
@@
 <net name="A0" class="0">
 <segment>
-<pinref part="JP_LEFT" gate="G$1" pin="5"/>
+<pinref part="ARDUINO_PRO_MINI_LEFT" gate="G$1" pin="5"/>
 <wire x1="60.96" y1="86.36" x2="48.26" y2="86.36" width="0.1524" layer="91"/>
 <label x="48.26" y="86.36" size="1.778" layer="95"/>
@@
 <net name="G13" class="0">
 <segment>
-<pinref part="JP_LEFT" gate="G$1" pin="4"/>
+<pinref part="ARDUINO_PRO_MINI_LEFT" gate="G$1" pin="4"/>
 <wire x1="60.96" y1="88.9" x2="35.56" y2="88.9" width="0.1524" layer="91"/>
 <label x="30.48" y="88.9" size="1.778" layer="95"/>
@@
 <net name="G12" class="0">
 <segment>
-<pinref part="JP_LEFT" gate="G$1" pin="3"/>
+<pinref part="ARDUINO_PRO_MINI_LEFT" gate="G$1" pin="3"/>
 <wire x1="60.96" y1="91.44" x2="48.26" y2="91.44" width="0.1524" layer="91"/>
 <label x="50.8" y="91.44" size="1.778" layer="95"/>
@@
 <net name="G11" class="0">
 <segment>
-<pinref part="JP_LEFT" gate="G$1" pin="2"/>
+<pinref part="ARDUINO_PRO_MINI_LEFT" gate="G$1" pin="2"/>
 <wire x1="60.96" y1="93.98" x2="35.56" y2="93.98" width="0.1524" layer="91"/>
 <label x="38.1" y="93.98" size="1.778" layer="95"/>
@@
 <net name="G10" class="0">
 <segment>
-<pinref part="JP_LEFT" gate="G$1" pin="1"/>
+<pinref part="ARDUINO_PRO_MINI_LEFT" gate="G$1" pin="1"/>
 <wire x1="60.96" y1="96.52" x2="48.26" y2="96.52" width="0.1524" layer="91"/>
 <label x="48.26" y="96.52" size="1.778" layer="95"/>
@@
 <net name="TXO" class="0">
 <segment>
-<pinref part="JP_RIGHT" gate="G$1" pin="12"/>
+<pinref part="ARDUINO_PRO_MINI_RIGHT" gate="G$1" pin="12"/>
 <wire x1="111.76" y1="68.58" x2="88.9" y2="68.58" width="0.1524" layer="91"/>
 <label x="88.9" y="68.58" size="1.778" layer="95"/>
@@
 <net name="RXI" class="0">
 <segment>
-<pinref part="JP_RIGHT" gate="G$1" pin="11"/>
+<pinref part="ARDUINO_PRO_MINI_RIGHT" gate="G$1" pin="11"/>
 <wire x1="111.76" y1="71.12" x2="99.06" y2="71.12" width="0.1524" layer="91"/>
 <label x="99.06" y="71.12" size="1.778" layer="95"/>
@@
 <net name="G2" class="0">
 <segment>
-<pinref part="JP_RIGHT" gate="G$1" pin="8"/>
+<pinref part="ARDUINO_PRO_MINI_RIGHT" gate="G$1" pin="8"/>
 <wire x1="111.76" y1="78.74" x2="91.44" y2="78.74" width="0.1524" layer="91"/>
 <label x="93.98" y="78.74" size="1.778" layer="95"/>
@@
 <net name="G3" class="0">
 <segment>
-<pinref part="JP_RIGHT" gate="G$1" pin="7"/>
+<pinref part="ARDUINO_PRO_MINI_RIGHT" gate="G$1" pin="7"/>
 <wire x1="111.76" y1="81.28" x2="99.06" y2="81.28" width="0.1524" layer="91"/>
 <label x="101.6" y="81.28" size="1.778" layer="95"/>
@@
 <net name="G4" class="0">
 <segment>
-<pinref part="JP_RIGHT" gate="G$1" pin="6"/>
+<pinref part="ARDUINO_PRO_MINI_RIGHT" gate="G$1" pin="6"/>
 <wire x1="111.76" y1="83.82" x2="91.44" y2="83.82" width="0.1524" layer="91"/>
 <label x="93.98" y="83.82" size="1.778" layer="95"/>
@@
 <net name="G5" class="0">
 <segment>
-<pinref part="JP_RIGHT" gate="G$1" pin="5"/>
+<pinref part="ARDUINO_PRO_MINI_RIGHT" gate="G$1" pin="5"/>
 <wire x1="111.76" y1="86.36" x2="99.06" y2="86.36" width="0.1524" layer="91"/>
 <label x="99.06" y="86.36" size="1.778" layer="95"/>
@@
 <net name="G6" class="0">
 <segment>
-<pinref part="JP_RIGHT" gate="G$1" pin="4"/>
+<pinref part="ARDUINO_PRO_MINI_RIGHT" gate="G$1" pin="4"/>
 <wire x1="111.76" y1="88.9" x2="91.44" y2="88.9" width="0.1524" layer="91"/>
 <label x="91.44" y="88.9" size="1.778" layer="95"/>
@@
 <net name="G7" class="0">
 <segment>
-<pinref part="JP_RIGHT" gate="G$1" pin="3"/>
+<pinref part="ARDUINO_PRO_MINI_RIGHT" gate="G$1" pin="3"/>
 <wire x1="111.76" y1="91.44" x2="99.06" y2="91.44" width="0.1524" layer="91"/>
 <label x="99.06" y="91.44" size="1.778" layer="95"/>
@@
 <net name="G8" class="0">
 <segment>
-<pinref part="JP_RIGHT" gate="G$1" pin="2"/>
+<pinref part="ARDUINO_PRO_MINI_RIGHT" gate="G$1" pin="2"/>
 <wire x1="111.76" y1="93.98" x2="91.44" y2="93.98" width="0.1524" layer="91"/>
 <label x="91.44" y="93.98" size="1.778" layer="95"/>
@@
 <net name="G9" class="0">
 <segment>
-<pinref part="JP_RIGHT" gate="G$1" pin="1"/>
+<pinref part="ARDUINO_PRO_MINI_RIGHT" gate="G$1" pin="1"/>
 <wire x1="111.76" y1="96.52" x2="99.06" y2="96.52" width="0.1524" layer="91"/>
 <label x="101.6" y="96.52" size="1.778" layer="95"/>
@@
 </segment>
 <segment>
-<pinref part="JP2" gate="G$1" pin="1"/>
-<wire x1="7.62" y1="60.96" x2="25.4" y2="60.96" width="0.1524" layer="91"/>
-<label x="20.32" y="60.96" size="1.778" layer="95"/>
+<pinref part="JP_I2C_OLED_SSD1306" gate="A" pin="4"/>
+<wire x1="38.1" y1="40.64" x2="17.78" y2="40.64" width="0.1524" layer="91"/>
+<label x="17.78" y="40.64" size="1.778" layer="95"/>
 </segment>
 </net>
@@
 <label x="83.82" y="53.34" size="1.778" layer="95" rot="R90"/>
 </segment>
-</net>
+<segment>
+<pinref part="JP_I2C_OLED_SSD1306" gate="A" pin="3"/>
+<wire x1="38.1" y1="43.18" x2="17.78" y2="43.18" width="0.1524" layer="91"/>
+<label x="15.24" y="43.18" size="1.778" layer="95"/>
+</segment>
+</net>
