File: USB.BusinessCard/bu/USB.BusinessCard.brd (EAGLE design)
At the start: 30 x 90 mm, 6 parts

Commit message: Update firmware for Usb Business Card
Parts:
- moved JP_PROGRAMMING 4.00 mm to (2.00, 67.5)
Connections:
- new net GND2: ARDUINO_PRO_MINI_RIGHT.9
- new net RST_2: ARDUINO_PRO_MINI_RIGHT.10
- net GND: no longer ARDUINO_PRO_MINI_RIGHT.9
- net RST: no longer ARDUINO_PRO_MINI_RIGHT.10
Other:
- board text added: "PCB v1 - 2019.10"
- board text added: "https://bit.ly/2J5fCQa"
- board text removed: "PCB v 2019.10"
Changed lines of the file:
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@@
 Business Card</text>
 <text x="27.5" y="48.5" size="2.54" layer="26" rot="MR270" align="center">www.FredericTorres.com</text>
-<text x="15.7" y="72" size="1.27" layer="26" rot="MR90" align="center">PCB v 2019.10</text>
+<text x="19.7" y="72" size="1.4224" layer="26" rot="MR90" align="center">https://bit.ly/2J5fCQa</text>
 <wire x1="21" y1="9" x2="21" y2="0" width="0.4064" layer="20"/>
 <wire x1="21" y1="0" x2="9" y2="0" width="0.4064" layer="20"/>
@@
 <text x="4.5" y="26.2" size="1.016" layer="25" rot="R180" align="center">A3</text>
 <text x="26" y="20.7" size="1.016" layer="25" rot="R180" align="center">*RST</text>
-<text x="26" y="23.7" size="1.016" layer="25" rot="R180" align="center">*GND</text>
+<text x="26" y="23.7" size="1.016" layer="25" rot="R180" align="center">GND</text>
 <text x="4.5" y="28.7" size="1.016" layer="25" rot="R180" align="center">A2</text>
 <text x="4.5" y="31.2" size="1.016" layer="25" rot="R180" align="center">A1</text>
@@
 <text x="26" y="16.2" size="1.016" layer="25" rot="R180" align="center">TXO</text>
 <text x="4.5" y="16.2" size="1.016" layer="25" rot="R180" align="center">RAW</text>
-<text x="5.5" y="57.2" size="1.016" layer="25" rot="R180" align="center">GND</text>
-<text x="5.5" y="59.7" size="1.016" layer="25" rot="R180" align="center">VCC</text>
-<text x="5.5" y="62.2" size="1.016" layer="25" rot="R180" align="center">RST</text>
-<text x="7" y="64.7" size="1.016" layer="25" rot="R180" align="center">G13_SCK</text>
-<text x="7.5" y="67.2" size="1.016" layer="25" rot="R180" align="center">G12_MISO</text>
-<text x="7.5" y="69.7" size="1.016" layer="25" rot="R180" align="center">G11_MOSI</text>
+<text x="5.5" y="61.2" size="1.016" layer="25" rot="R180" align="center">GND</text>
+<text x="5.5" y="63.7" size="1.016" layer="25" rot="R180" align="center">VCC</text>
+<text x="5.5" y="66.2" size="1.016" layer="25" rot="R180" align="center">RST</text>
+<text x="7" y="68.7" size="1.016" layer="25" rot="R180" align="center">G13_SCK</text>
+<text x="7.5" y="71.2" size="1.016" layer="25" rot="R180" align="center">G12_MISO</text>
+<text x="7.5" y="73.7" size="1.016" layer="25" rot="R180" align="center">G11_MOSI</text>
 <text x="14.5" y="12.5" size="1.4224" layer="25" rot="R180" align="center">www.FredericTorres.com</text>
 <text x="25.6" y="71.1" size="2.54" layer="25" rot="R90" align="center">Frederic Torres
 Business Card</text>
 <text x="14.6" y="12.4" size="1.4224" layer="25" rot="R180" align="center">www.FredericTorres.com</text>
+<text x="10.7" y="72" size="1.27" layer="26" rot="MR90" align="center">PCB v1 - 2019.10</text>
 </plain>
 <attributes>
@@
 <attribute name="VALUE" x="20.08" y="56.175" size="1.27" layer="27" rot="R180"/>
 </element>
-<element name="JP_PROGRAMMING" library="adafruit" package="1X06" value="" x="2" y="63.5" smashed="yes" rot="R90">
-<attribute name="NAME" x="1.6712" y="78.3038" size="1.016" layer="25" ratio="10" rot="R90" align="center"/>
-<attribute name="VALUE" x="5.175" y="55.88" size="1.27" layer="27" rot="R90"/>
+<element name="JP_PROGRAMMING" library="adafruit" package="1X06" value="" x="2" y="67.5" smashed="yes" rot="R90">
+<attribute name="NAME" x="1.6712" y="82.3038" size="1.016" layer="25" ratio="10" rot="R90" align="center"/>
+<attribute name="VALUE" x="5.175" y="59.88" size="1.27" layer="27" rot="R90"/>
 </element>
 </elements>
@@
 <contactref element="JP1" pad="GND"/>
 <contactref element="ARDUINO_PRO_MINI_LEFT" pad="11"/>
-<contactref element="ARDUINO_PRO_MINI_RIGHT" pad="9"/>
 <contactref element="JP_I2C_OLED_SSD1306" pad="1"/>
 <contactref element="JP_PROGRAMMING" pad="1"/>
-<wire x1="2" y1="57.15" x2="18.81" y2="53" width="0" layer="19" extent="1-1"/>
-<wire x1="22.7" y1="23.65" x2="18.81" y2="53" width="0" layer="19" extent="1-1"/>
-<wire x1="8" y1="18.57" x2="22.7" y2="23.65" width="0" layer="19" extent="1-1"/>
+<wire x1="2" y1="61.15" x2="18.81" y2="53" width="0" layer="19" extent="1-1"/>
+<wire x1="8" y1="18.57" x2="18.81" y2="53" width="0" layer="19" extent="1-1"/>
 <wire x1="11.5" y1="4.8" x2="8" y2="18.57" width="0" layer="19" extent="1-1"/>
 </signal>
@@
 <contactref element="JP_I2C_OLED_SSD1306" pad="2"/>
 <contactref element="JP_PROGRAMMING" pad="2"/>
-<wire x1="2" y1="59.69" x2="16.27" y2="53" width="0" layer="19" extent="1-1"/>
+<wire x1="2" y1="63.69" x2="16.27" y2="53" width="0" layer="19" extent="1-1"/>
 <wire x1="8" y1="23.65" x2="16.27" y2="53" width="0" layer="19" extent="1-1"/>
 <wire x1="18.5" y1="4.8" x2="8" y2="23.65" width="0" layer="19" extent="1-1"/>
@@
 <signal name="RST">
 <contactref element="ARDUINO_PRO_MINI_LEFT" pad="10"/>
-<contactref element="ARDUINO_PRO_MINI_RIGHT" pad="10"/>
 <contactref element="JP_PROGRAMMING" pad="3"/>
-<wire x1="8" y1="21.11" x2="2" y2="62.23" width="0" layer="19" extent="1-1"/>
-<wire x1="22.7" y1="21.11" x2="8" y2="21.11" width="0" layer="19" extent="1-1"/>
+<wire x1="8" y1="21.11" x2="2" y2="66.23" width="0" layer="19" extent="1-1"/>
 </signal>
 <signal name="A3">
@@
 <contactref element="ARDUINO_PRO_MINI_LEFT" pad="4"/>
 <contactref element="JP_PROGRAMMING" pad="4"/>
-<wire x1="8" y1="36.35" x2="2" y2="64.77" width="0" layer="19" extent="1-1"/>
+<wire x1="8" y1="36.35" x2="2" y2="68.77" width="0" layer="19" extent="1-1"/>
 </signal>
 <signal name="G12_MISO">
 <contactref element="ARDUINO_PRO_MINI_LEFT" pad="3"/>
 <contactref element="JP_PROGRAMMING" pad="5"/>
-<wire x1="8" y1="38.89" x2="2" y2="67.31" width="0" layer="19" extent="1-1"/>
+<wire x1="8" y1="38.89" x2="2" y2="71.31" width="0" layer="19" extent="1-1"/>
 </signal>
 <signal name="G11_MOSI">
 <contactref element="ARDUINO_PRO_MINI_LEFT" pad="2"/>
 <contactref element="JP_PROGRAMMING" pad="6"/>
-<wire x1="8" y1="41.43" x2="2" y2="69.85" width="0" layer="19" extent="1-1"/>
+<wire x1="8" y1="41.43" x2="2" y2="73.85" width="0" layer="19" extent="1-1"/>
 </signal>
 <signal name="G10">
@@
 <contactref element="JP_TOP" pad="4"/>
 </signal>
+<signal name="RST_2">
+<contactref element="ARDUINO_PRO_MINI_RIGHT" pad="10"/>
+</signal>
+<signal name="GND2">
+<contactref element="ARDUINO_PRO_MINI_RIGHT" pad="9"/>
+</signal>
 </signals>
