File: EXTENSIONS/Analog/OneLedBlinker/bu/OneLedBlinker.sch (EAGLE design)
At the start: 9 parts, among them X1 USB-A

Commit message: Revisit One Led Blinker pcb
Parts:
- removed GND: GND, adafruit:PINHD-1X1
Connections:
- net N$4: no longer GND.1
Changed lines of the file:
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@@
 <part name="C1_100UF" library="adafruit" deviceset="C-US" device="025-030X050"/>
 <part name="R1M" library="adafruit" deviceset="R-US_" device="0207/10"/>
-<part name="GND" library="adafruit" deviceset="PINHD-1X1" device="" value="GND"/>
 </parts>
 <sheets>
@@
 <instance part="C1_100UF" gate="G$1" x="50.8" y="83.82" rot="R90"/>
 <instance part="R1M" gate="G$1" x="33.02" y="63.5" rot="R90"/>
-<instance part="GND" gate="G$1" x="101.6" y="99.06" rot="R90"/>
 </instances>
 <busses>
@@
 <wire x1="68.58" y1="58.42" x2="68.58" y2="60.96" width="0.1524" layer="91"/>
 <junction x="68.58" y="60.96"/>
-<pinref part="GND" gate="G$1" pin="1"/>
-<wire x1="101.6" y1="96.52" x2="101.6" y2="88.9" width="0.1524" layer="91"/>
-<junction x="101.6" y="88.9"/>
 </segment>
 </net>
