File: EXTENSIONS/Analog/fCPU.Controller1/fCPU.Controller1.sch (EAGLE design)
At the start: 8 parts, among them X1 USB-A

Commit message: Revisit One Led Blinker pcb
Parts:
- removed 2N3904_NPN: 2N3904, transistor:2N3904
- removed 2N3906_PNP: 2N3906, transistor-pnp:2N3906
- removed C1_100UF: (no value), adafruit:C-US025-030X050
- removed LED1: (no value), adafruit:LED5MM
- removed R10K, R1M, R22: (no value), adafruit:R-US_0207/10
- removed X1: USB-A, adafruit:USB-A
- added EXTERNAL_CONTROL_OUTPUT: (no value), adafruit:PINHD-1X12
- added IC1: 4017N, 40xx:4017N
- added JP_CLOCK_IN, OUTPUTS: (no value), pinhead:PINHD-1X4
- added LED_CLOCK: (no value), adafruit:LEDSMT1206
- added RESET_PROGRAM: (no value), switch-omron:10-XX
- added RESISTOR_SWITCHES: (no value), resistor-sip:4610X
- added R_100_O: (no value), adafruit:R-US_R1206
Connections:
- removed net N$1: 2N3906_PNP.E, R22.2, X1.VBUS
- removed net N$2: 2N3904_NPN.C, C1_100UF.2, R22.1
- removed net N$3: 2N3904_NPN.E, LED1.A
- removed net N$4: LED1.C, R1M.1, X1.GND
- removed net N$5: 2N3906_PNP.B, C1_100UF.1, R1M.2
- removed net N$6: 2N3906_PNP.C, R10K.1
- removed net N$7: 2N3904_NPN.B, R10K.2
- new net GND: IC1A.ENA, JP_CLOCK_IN.1, OUTPUTS.1, RESISTOR_SWITCHES.1
- new net LED_CLOCK_TO_GND: LED_CLOCK.C, RESISTOR_SWITCHES.9
- new net REGISTER_1_CLK: EXTERNAL_CONTROL_OUTPUT.9, IC1A.Q1
- new net REGISTER_1_CLR: EXTERNAL_CONTROL_OUTPUT.10
- new net REGISTER_1_IN_BIT_0: EXTERNAL_CONTROL_OUTPUT.1
- new net REGISTER_1_IN_BIT_1: EXTERNAL_CONTROL_OUTPUT.2
- new net REGISTER_1_IN_BIT_2: EXTERNAL_CONTROL_OUTPUT.3
- new net REGISTER_1_IN_BIT_3: EXTERNAL_CONTROL_OUTPUT.4
- new net REGISTER_2_CLK: EXTERNAL_CONTROL_OUTPUT.11
- new net REGISTER_2_CLR: EXTERNAL_CONTROL_OUTPUT.12
- new net REGISTER_2_IN_BIT_0: EXTERNAL_CONTROL_OUTPUT.5
- new net REGISTER_2_IN_BIT_1: EXTERNAL_CONTROL_OUTPUT.6
- new net REGISTER_2_IN_BIT_2: EXTERNAL_CONTROL_OUTPUT.7
- new net REGISTER_2_IN_BIT_3: EXTERNAL_CONTROL_OUTPUT.8
- new net TMR555_OUTPUT: IC1A.CLK, JP_CLOCK_IN.3, LED_CLOCK.A, OUTPUTS.3
- new net TMR555_OUTPUT_REVERSE: JP_CLOCK_IN.4, OUTPUTS.4
- new net VCC: JP_CLOCK_IN.2, OUTPUTS.2
