File: EXTENSIONS/Analog/fCPU.Controller1/bu/fCPU.Controller1.sch (EAGLE design)
At the start: 8 parts, among them X1 USB-A

Commit message: Revisit One Led Blinker pcb
Parts:
- removed 2N3904_NPN: 2N3904, transistor:2N3904
- removed 2N3906_PNP: 2N3906, transistor-pnp:2N3906
- removed C1_100UF: (no value), adafruit:C-US025-030X050
- removed LED1: (no value), adafruit:LED5MM
- removed R10K, R1M, R22: (no value), adafruit:R-US_0207/10
- removed X1: USB-A, adafruit:USB-A
- added ADDER_74LS283N: 74LS283N, 74xx-us:74LS283N
- added CLEAR_REGISTER_1, CLEAR_REGISTER_2, CLOCK_REGISTER_1, CLOCK_REGISTER_2: (no value), switch-omron:10-XX
- added DIGIT_0_ANODE: (no value), special:7SEG-CA
- added DISPLAY_DRIVER_74LS47: 74LS47N, 74xx-us:74LS47N
- added EXTERNAL_CONTROL_INPUT: (no value), adafruit:PINHD-1X12
- added INPUT_DEVICE_1, INPUT_DEVICE_2: (no value), special:SW_DIP-4
- added JP_CLOCK_IN, OUTPUTS: (no value), pinhead:PINHD-1X4
- added LED_POWER: (no value), adafruit:LEDSMT1206
- added REGISTER_1_SN74LS273, REGISTER_2_SN74LS273: 74273N, 74xx-us:74273N
- added RESISTOR_INPUT_DEVICES, RESISTOR_SWITCHES: (no value), resistor-sip:4610X
- added R_100_O: (no value), adafruit:R-US_R1206
Connections:
- removed net N$2: 2N3904_NPN.C, C1_100UF.2, R22.1
- removed net N$3: 2N3904_NPN.E, LED1.A
- removed net N$4: LED1.C, R1M.1, X1.GND
- removed net N$5: 2N3906_PNP.B, C1_100UF.1, R1M.2
- removed net N$6: 2N3906_PNP.C, R10K.1
- removed net N$7: 2N3904_NPN.B, R10K.2
- new net CLEAR_REGISTER_1_TO_GND: CLEAR_REGISTER_1.S, RESISTOR_SWITCHES.4
- new net CLEAR_REGISTER_2_TO_GND: CLEAR_REGISTER_2.S, RESISTOR_SWITCHES.5
- new net DTA_BUS_0: ADDER_74LS283NA.S1, DISPLAY_DRIVER_74LS47G$1.IA
- new net DTA_BUS_1: ADDER_74LS283NA.S2, DISPLAY_DRIVER_74LS47G$1.IB
- new net DTA_BUS_2: ADDER_74LS283NA.S3, DISPLAY_DRIVER_74LS47G$1.IC
- new net DTA_BUS_3: ADDER_74LS283NA.S4, DISPLAY_DRIVER_74LS47G$1.ID
- new net GND: ADDER_74LS283NA.C0, JP_CLOCK_IN.1, OUTPUTS.1, REGISTER_1_SN74LS273A.D5, REGISTER_1_SN74LS273A.D6, REGISTER_1_SN74LS273A.D7, REGISTER_1_SN74LS273A.D8, REGISTER_2_SN74LS273A.D5, REGISTER_2_SN74LS273A.D6, REGISTER_2_SN74LS273A.D7, REGISTER_2_SN74LS273A.D8, RESISTOR_INPUT_DEVICES.1, RESISTOR_SWITCHES.1
- new net LED_POWER_TO_GND: LED_POWER.C, RESISTOR_SWITCHES.9
- new net REGISTER_1_CLK: CLOCK_REGISTER_1.P1, EXTERNAL_CONTROL_INPUT.9, REGISTER_1_SN74LS273A.CLK, RESISTOR_SWITCHES.2
- new net REGISTER_1_CLR: CLEAR_REGISTER_1.P1, EXTERNAL_CONTROL_INPUT.10, REGISTER_1_SN74LS273A.CLR
- new net REGISTER_1_IN_BIT_0: EXTERNAL_CONTROL_INPUT.1, INPUT_DEVICE_1.1, REGISTER_1_SN74LS273A.D1, RESISTOR_INPUT_DEVICES.2
- new net REGISTER_1_IN_BIT_1: EXTERNAL_CONTROL_INPUT.2, INPUT_DEVICE_1.2, REGISTER_1_SN74LS273A.D2, RESISTOR_INPUT_DEVICES.3
- new net REGISTER_1_IN_BIT_2: EXTERNAL_CONTROL_INPUT.3, INPUT_DEVICE_1.3, REGISTER_1_SN74LS273A.D3, RESISTOR_INPUT_DEVICES.4
- new net REGISTER_1_IN_BIT_3: EXTERNAL_CONTROL_INPUT.4, INPUT_DEVICE_1.4, REGISTER_1_SN74LS273A.D4, RESISTOR_INPUT_DEVICES.5
- new net REGISTER_1_OUT_BIT_0: ADDER_74LS283NA.A1, REGISTER_1_SN74LS273A.Q1
- new net REGISTER_1_OUT_BIT_1: ADDER_74LS283NA.A2, REGISTER_1_SN74LS273A.Q2
- new net REGISTER_1_OUT_BIT_2: ADDER_74LS283NA.A3, REGISTER_1_SN74LS273A.Q3
- new net REGISTER_1_OUT_BIT_3: ADDER_74LS283NA.A4, REGISTER_1_SN74LS273A.Q4
- new net REGISTER_2_CLK: CLOCK_REGISTER_2.P1, EXTERNAL_CONTROL_INPUT.11, REGISTER_2_SN74LS273A.CLK, RESISTOR_SWITCHES.3
- new net REGISTER_2_CLR: CLEAR_REGISTER_2.P1, EXTERNAL_CONTROL_INPUT.12, REGISTER_2_SN74LS273A.CLR
- new net REGISTER_2_IN_BIT_0: EXTERNAL_CONTROL_INPUT.5, INPUT_DEVICE_2.1, REGISTER_2_SN74LS273A.D1, RESISTOR_INPUT_DEVICES.6
- new net REGISTER_2_IN_BIT_1: EXTERNAL_CONTROL_INPUT.6, INPUT_DEVICE_2.2, REGISTER_2_SN74LS273A.D2, RESISTOR_INPUT_DEVICES.7
- new net REGISTER_2_IN_BIT_2: EXTERNAL_CONTROL_INPUT.7, INPUT_DEVICE_2.3, REGISTER_2_SN74LS273A.D3, RESISTOR_INPUT_DEVICES.8
- new net REGISTER_2_IN_BIT_3: EXTERNAL_CONTROL_INPUT.8, INPUT_DEVICE_2.4, REGISTER_2_SN74LS273A.D4, RESISTOR_INPUT_DEVICES.9
- new net REGISTER_2_OUT_BIT_0: ADDER_74LS283NA.B1, REGISTER_2_SN74LS273A.Q1
- new net REGISTER_2_OUT_BIT_1: ADDER_74LS283NA.B2, REGISTER_2_SN74LS273A.Q2
- new net REGISTER_2_OUT_BIT_2: ADDER_74LS283NA.B3, REGISTER_2_SN74LS273A.Q3
- new net REGISTER_2_OUT_BIT_3: ADDER_74LS283NA.B4, REGISTER_2_SN74LS273A.Q4
- new net SEG_1_DA: DIGIT_0_ANODE.A, DISPLAY_DRIVER_74LS47G$1.A
- new net SEG_1_DB: DIGIT_0_ANODE.B, DISPLAY_DRIVER_74LS47G$1.B
- new net SEG_1_DC: DIGIT_0_ANODE.C, DISPLAY_DRIVER_74LS47G$1.C
- new net SEG_1_DD: DIGIT_0_ANODE.D, DISPLAY_DRIVER_74LS47G$1.D
- new net SEG_1_DE: DIGIT_0_ANODE.E, DISPLAY_DRIVER_74LS47G$1.E
- new net SEG_1_DF: DIGIT_0_ANODE.F, DISPLAY_DRIVER_74LS47G$1.F
- new net SEG_1_DG: DIGIT_0_ANODE.G, DISPLAY_DRIVER_74LS47G$1.G
- new net TMR555_OUTPUT: JP_CLOCK_IN.3, OUTPUTS.3
- new net TMR555_OUTPUT_REVERSE: JP_CLOCK_IN.4, OUTPUTS.4
- new net VCC: CLOCK_REGISTER_1.S, CLOCK_REGISTER_2.S, DISPLAY_DRIVER_74LS47G$1.BI/RBO, DISPLAY_DRIVER_74LS47G$1.LT, DISPLAY_DRIVER_74LS47G$1.RBI, INPUT_DEVICE_1.5, INPUT_DEVICE_1.6, INPUT_DEVICE_1.7, INPUT_DEVICE_1.8, INPUT_DEVICE_2.5, INPUT_DEVICE_2.6, INPUT_DEVICE_2.7, INPUT_DEVICE_2.8, JP_CLOCK_IN.2, LED_POWER.A, OUTPUTS.2, R_100_O.2
- net N$1: now also DIGIT_0_ANODE.CA2, R_100_O.1; no longer 2N3906_PNP.E, R22.2, X1.VBUS
