File: EXTENSIONS/Analog/4017-7Segment/v2.Bug.UseSegmentGAndShouldNot/4017-7Segment.brd (EAGLE design)
At the start: 53 x 43 mm, 7 parts

Commit message: Fix bug in 4017-7Segment v2
Connections:
- net RESET: no longer 4017BE.5
- net SEG_G: now also 4017BE.5
Changed lines of the file:
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@@
 <layer number="23" name="tOrigins" color="15" fill="1" visible="yes" active="yes"/>
 <layer number="24" name="bOrigins" color="15" fill="1" visible="yes" active="yes"/>
-<layer number="25" name="tNames" color="7" fill="1" visible="yes" active="yes"/>
-<layer number="26" name="bNames" color="7" fill="1" visible="no" active="yes"/>
+<layer number="25" name="tNames" color="7" fill="1" visible="no" active="yes"/>
+<layer number="26" name="bNames" color="7" fill="1" visible="yes" active="yes"/>
 <layer number="27" name="tValues" color="7" fill="1" visible="no" active="yes"/>
 <layer number="28" name="bValues" color="7" fill="1" visible="no" active="yes"/>
@@
 <signal name="SEG_G">
 <contactref element="U$1" pad="10"/>
+<contactref element="4017BE" pad="5"/>
+<wire x1="6.42" y1="51.12" x2="38.77" y2="42.69" width="0" layer="19" extent="1-1"/>
 </signal>
 <signal name="SEG_DP">
@@
 <contactref element="4017BE" pad="6"/>
 <contactref element="4017BE" pad="15"/>
-<contactref element="4017BE" pad="5"/>
-<wire x1="38.77" y1="42.69" x2="41.31" y2="42.69" width="0" layer="19" extent="1-1"/>
-<wire x1="31.15" y1="50.31" x2="38.77" y2="42.69" width="0" layer="19" extent="1-1"/>
+<wire x1="31.15" y1="50.31" x2="41.31" y2="42.69" width="0" layer="19" extent="1-1"/>
 </signal>
 <signal name="N$1">
