File: EXTENSIONS/Analog/UpTo11/FrontPanel/v1/UpTo11.FrontPanel.brd (EAGLE design)
At the start: 68 x 58 mm, 6 parts

Commit message: Fix bugs in UpTo11, 2 baord
Parts:
- moved FRONT_PANEL_INTERFACE 1.50 mm to (36.5, 14.5)
Other:
- outline, holes or cut-outs redrawn
Changed lines of the file:
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@@
 <text x="30" y="21.5" size="1.27" layer="26" rot="MR90" align="center">POT_OUT</text>
 <hole x="26" y="39.5" drill="7"/>
-<rectangle x1="17.5" y1="38" x2="18.7" y2="40.6" layer="46"/>
+<rectangle x1="17" y1="38" x2="18.2" y2="40.6" layer="46"/>
 <rectangle x1="19.42518125" y1="27.08558125" x2="19.67918125" y2="27.17041875" layer="21"/>
 <rectangle x1="32.717" y1="27.08558125" x2="32.80081875" y2="27.17041875" layer="21"/>
@@
 </autorouter>
 <elements>
-<element name="FRONT_PANEL_INTERFACE" library="adafruit" package="1X06" value="" x="35" y="14.5" smashed="yes" rot="R180">
-<attribute name="VALUE" x="42.62" y="17.675" size="1.27" layer="27" rot="R180"/>
+<element name="FRONT_PANEL_INTERFACE" library="adafruit" package="1X06" value="" x="36.5" y="14.5" smashed="yes" rot="R180">
+<attribute name="VALUE" x="44.12" y="17.675" size="1.27" layer="27" rot="R180"/>
 </element>
 <element name="POWER" library="adafruit" package="1206" value="" x="63" y="23" smashed="yes">
@@
 <contactref element="FRONT_PANEL_INTERFACE" pad="4"/>
 <contactref element="FLASH_LED" pad="A"/>
-<wire x1="56.91521875" y1="51.206278125" x2="33.73" y2="14.5" width="0" layer="19" extent="1-1"/>
+<wire x1="56.91521875" y1="51.206278125" x2="35.23" y2="14.5" width="0" layer="19" extent="1-1"/>
 </signal>
 <signal name="GND_EX">
@@
 <contactref element="POT_GND_(LEFT)" pad="2"/>
 <wire x1="64.422" y1="23" x2="59.45521875" y2="51.206278125" width="0" layer="19" extent="1-1"/>
-<wire x1="41.35" y1="14.5" x2="64.422" y2="23" width="0" layer="19" extent="1-1"/>
-<wire x1="25" y1="19.238" x2="41.35" y2="14.5" width="0" layer="19" extent="1-1"/>
+<wire x1="42.85" y1="14.5" x2="64.422" y2="23" width="0" layer="19" extent="1-1"/>
+<wire x1="25" y1="19.238" x2="42.85" y2="14.5" width="0" layer="19" extent="1-1"/>
 </signal>
 <signal name="VCC">
@@
 <contactref element="FRONT_PANEL_INTERFACE" pad="3"/>
 <contactref element="POWER" pad="A"/>
-<wire x1="61.578" y1="23" x2="36.27" y2="14.5" width="0" layer="19" extent="1-1"/>
+<wire x1="61.578" y1="23" x2="37.77" y2="14.5" width="0" layer="19" extent="1-1"/>
 </signal>
 <signal name="POT_IN">
 <contactref element="FRONT_PANEL_INTERFACE" pad="5"/>
 <contactref element="POT_IN_(MIDDLE)" pad="2"/>
-<wire x1="17" y1="19.238" x2="31.19" y2="14.5" width="0" layer="19" extent="1-1"/>
+<wire x1="17" y1="19.238" x2="32.69" y2="14.5" width="0" layer="19" extent="1-1"/>
 </signal>
 <signal name="POT_OUT">
 <contactref element="FRONT_PANEL_INTERFACE" pad="6"/>
 <contactref element="POT_OUT_(RIGHT)" pad="2"/>
-<wire x1="8" y1="19.238" x2="28.65" y2="14.5" width="0" layer="19" extent="1-1"/>
+<wire x1="8" y1="19.238" x2="30.15" y2="14.5" width="0" layer="19" extent="1-1"/>
 </signal>
 </signals>
