File: EXTENSIONS/Analog/CheetahBooster/v1/CheetahBooster.sch (EAGLE design)
At the start: 28 parts

Commit message: Update CheetahBoosyer v2
Parts:
- removed D10, D11, D12, D13, D14, D15, D16, D17, D18, D19, D20, D21: (no value), adafruit:DIODESMA
- added SJ1, SJ10, SJ11, SJ12, SJ14, SJ15, SJ16, SJ18, SJ19, SJ2, SJ20, SJ21, SJ22, SJ23, SJ3, SJ4, SJ5, SJ6, SJ7, SJ8, SJ9: (no value), microbuilder:SOLDERJUMPER
- D1, D2, D3, D4, D5, D6, D7, D8, D9: value (none) -> 1N821; device adafruit:DIODESMA -> diode:1N821
Connections:
- new net SEG_1_1: D2.C, SJ2.1, SJ4.1
- new net SEG_2_2: D3.C, SJ3.1, SJ5.1, SJ8.1
- new net SEG_3_3: D4.C, SJ10.1, SJ22.2, SJ6.1
- new net SEG_4_4: D5.C, SJ12.1, SJ23.2, SJ9.1
- new net SEG_5_5: D6.C, SJ11.1, SJ14.1, SJ7.1
- new net SEG_6_6: D7.C, SJ15.1, SJ18.1, SJ21.2
- new net SEG_7_7: D8.C, SJ16.1, SJ19.1
- new net SEG_8_8: D9.C, SJ20.1
- net LED_0: now also SJ1.2, SJ2.2, SJ22.1, SJ3.2; no longer D1.C, D2.C, D3.C, D4.C
- net LED_1: now also SJ23.1, SJ4.2, SJ5.2; no longer D5.C, D6.C, D7.C
- net LED_2: now also SJ6.2, SJ7.2; no longer D8.C, D9.C
- net LED_3: now also SJ8.2, SJ9.2; no longer D10.C, D11.C
- net LED_4: now also SJ10.2, SJ11.2, SJ21.1; no longer D12.C, D13.C, D14.C
- net LED_5: now also SJ12.2; no longer D15.C
- net LED_6: now also SJ14.2, SJ15.2, SJ16.2; no longer D16.C, D17.C, D18.C
- net LED_7: now also SJ18.2, SJ19.2, SJ20.2; no longer D19.C, D20.C, D21.C
- net SEG_0_0: now also D1.C, SJ1.1
- net SEG_1: no longer D5.A
- net SEG_2: no longer D10.A, D6.A
- net SEG_3: no longer D12.A, D8.A
- net SEG_4: now also D5.A; no longer D11.A, D15.A, D7.A
- net SEG_5: now also D6.A; no longer D13.A, D16.A, D9.A
- net SEG_6: now also D7.A; no longer D14.A, D17.A, D19.A
- net SEG_7: now also D8.A; no longer D18.A, D20.A
- net SEG_8: now also D9.A; no longer D21.A
